File: hardware/power.kicad_sch (KiCad schematic)
At the start: 28 parts, among them U2 LT3988, U3 RC4558

Commit message: workin away
Parts:
- C10, C11, C13, C15, C7: footprint (none) -> Capacitor_SMD:C_1206_3216Metric_Pad1.33x1.80mm_HandSolder
- C12, C14, C16, C17, C19, C5, C8, C9, R1, R2, R3, R4, R5, R6, R7: footprint (none) -> Capacitor_SMD:C_0805_2012Metric_Pad1.18x1.45mm_HandSolder
- C18: value (none) -> 470n; footprint (none) -> Capacitor_SMD:C_0805_2012Metric_Pad1.18x1.45mm_HandSolder
- C6: value (none) -> 4.7u; footprint (none) -> Capacitor_SMD:C_1206_3216Metric_Pad1.33x1.80mm_HandSolder
- D1, D2: value (none) -> PMEG100T10ELXD; footprint (none) -> Diode_SMD:D_SOD-323F
- L1, L2: value (none) -> 10u; footprint (none) -> Inductor_SMD:L_Taiyo-Yuden_MD-3030
- U3: footprint (none) -> Package_SO:SOIC-8-1EP_3.9x4.9mm_P1.27mm_EP2.514x3.2mm
Changed lines of the file:
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@@
     (property "Reference" "R5" (id 0) (at 119.38 90.17 90))
     (property "Value" "34k" (id 1) (at 119.38 92.71 90))
-    (property "Footprint" "" (id 2) (at 119.38 96.52 0)
+    (property "Footprint" "Capacitor_SMD:C_0805_2012Metric_Pad1.18x1.45mm_HandSolder" (id 2) (at 119.38 96.52 0)
       (effects (font (size 1.27 1.27)) hide)
     )
@@
       (effects (font (size 1.27 1.27)) (justify left))
     )
-    (property "Value" "" (id 1) (at 127 91.44 90)
-      (effects (font (size 1.27 1.27)) (justify left))
-    )
-    (property "Footprint" "" (id 2) (at 122.555 88.9 0)
+    (property "Value" "PMEG100T10ELXD" (id 1) (at 127 91.44 90)
+      (effects (font (size 1.27 1.27)) (justify left))
+    )
+    (property "Footprint" "Diode_SMD:D_SOD-323F" (id 2) (at 122.555 88.9 0)
       (effects (font (size 1.27 1.27)) hide)
     )
@@
     (property "Reference" "C17" (id 0) (at 119.38 104.14 90))
     (property "Value" "22p" (id 1) (at 119.38 106.68 90))
-    (property "Footprint" "" (id 2) (at 119.38 101.6 0)
+    (property "Footprint" "Capacitor_SMD:C_0805_2012Metric_Pad1.18x1.45mm_HandSolder" (id 2) (at 119.38 101.6 0)
       (effects (font (size 1.27 1.27)) hide)
     )
@@
       (effects (font (size 1.27 1.27)) (justify left))
     )
-    (property "Footprint" "" (id 2) (at 256.54 38.1 0)
+    (property "Footprint" "Package_SO:SOIC-8-1EP_3.9x4.9mm_P1.27mm_EP2.514x3.2mm" (id 2) (at 256.54 38.1 0)
       (effects (font (size 1.27 1.27)) hide)
     )
@@
       (effects (font (size 1.27 1.27)) (justify left))
     )
-    (property "Footprint" "" (id 2) (at 228.6 33.02 0)
+    (property "Footprint" "Capacitor_SMD:C_0805_2012Metric_Pad1.18x1.45mm_HandSolder" (id 2) (at 228.6 33.02 0)
       (effects (font (size 1.27 1.27)) hide)
     )
@@
     (property "Reference" "C16" (id 0) (at 116.84 68.58 90))
     (property "Value" "1n" (id 1) (at 119.38 68.58 90))
-    (property "Footprint" "" (id 2) (at 114.3 68.58 0)
+    (property "Footprint" "Capacitor_SMD:C_0805_2012Metric_Pad1.18x1.45mm_HandSolder" (id 2) (at 114.3 68.58 0)
       (effects (font (size 1.27 1.27)) hide)
     )
@@
     (in_bom yes) (on_board yes) (fields_autoplaced)
     (property "Reference" "L2" (id 0) (at 134.62 77.47 90))
-    (property "Value" "" (id 1) (at 134.62 80.01 90))
-    (property "Footprint" "" (id 2) (at 134.62 83.82 0)
+    (property "Value" "10u" (id 1) (at 134.62 80.01 90))
+    (property "Footprint" "Inductor_SMD:L_Taiyo-Yuden_MD-3030" (id 2) (at 134.62 83.82 0)
       (effects (font (size 1.27 1.27)) hide)
     )
@@
       (effects (font (size 1.27 1.27)) (justify right))
     )
-    (property "Footprint" "" (id 2) (at 109.22 104.14 0)
+    (property "Footprint" "Capacitor_SMD:C_0805_2012Metric_Pad1.18x1.45mm_HandSolder" (id 2) (at 109.22 104.14 0)
       (effects (font (size 1.27 1.27)) hide)
     )
@@
     (property "Reference" "R1" (id 0) (at 60.96 90.17 90))
     (property "Value" "150k" (id 1) (at 60.96 92.71 90))
-    (property "Footprint" "" (id 2) (at 60.96 96.52 0)
+    (property "Footprint" "Capacitor_SMD:C_0805_2012Metric_Pad1.18x1.45mm_HandSolder" (id 2) (at 60.96 96.52 0)
       (effects (font (size 1.27 1.27)) hide)
     )
@@
     (property "Reference" "C12" (id 0) (at 99.06 45.72 90))
     (property "Value" "22p" (id 1) (at 101.6 45.72 90))
-    (property "Footprint" "" (id 2) (at 96.52 45.72 0)
+    (property "Footprint" "Capacitor_SMD:C_0805_2012Metric_Pad1.18x1.45mm_HandSolder" (id 2) (at 96.52 45.72 0)
       (effects (font (size 1.27 1.27)) hide)
     )
@@
       (effects (font (size 1.27 1.27)) (justify left))
     )
-    (property "Value" "" (id 1) (at 53.34 153.6762 0)
-      (effects (font (size 1.27 1.27)) (justify left))
-    )
-    (property "Footprint" "" (id 2) (at 50.8 152.4 0)
+    (property "Value" "4.7u" (id 1) (at 53.34 153.6762 0)
+      (effects (font (size 1.27 1.27)) (justify left))
+    )
+    (property "Footprint" "Capacitor_SMD:C_1206_3216Metric_Pad1.33x1.80mm_HandSolder" (id 2) (at 50.8 152.4 0)
       (effects (font (size 1.27 1.27)) hide)
     )
@@
     (property "Reference" "C14" (id 0) (at 111.76 83.82 90))
     (property "Value" "220n" (id 1) (at 114.3 83.82 90))
-    (property "Footprint" "" (id 2) (at 109.22 83.82 0)
+    (property "Footprint" "Capacitor_SMD:C_0805_2012Metric_Pad1.18x1.45mm_HandSolder" (id 2) (at 109.22 83.82 0)
       (effects (font (size 1.27 1.27)) hide)
     )
@@
       (effects (font (size 1.27 1.27)) (justify left))
     )
-    (property "Footprint" "" (id 2) (at 76.2 152.4 0)
+    (property "Footprint" "Capacitor_SMD:C_1206_3216Metric_Pad1.33x1.80mm_HandSolder" (id 2) (at 76.2 152.4 0)
       (effects (font (size 1.27 1.27)) hide)
     )
@@
       (effects (font (size 1.27 1.27)) (justify right))
     )
-    (property "Footprint" "" (id 2) (at 68.58 104.14 0)
+    (property "Footprint" "Capacitor_SMD:C_0805_2012Metric_Pad1.18x1.45mm_HandSolder" (id 2) (at 68.58 104.14 0)
       (effects (font (size 1.27 1.27)) hide)
     )
@@
       (effects (font (size 1.27 1.27)) (justify left))
     )
-    (property "Footprint" "" (id 2) (at 60.96 152.4 0)
+    (property "Footprint" "Capacitor_SMD:C_1206_3216Metric_Pad1.33x1.80mm_HandSolder" (id 2) (at 60.96 152.4 0)
       (effects (font (size 1.27 1.27)) hide)
     )
@@
     (property "Reference" "C5" (id 0) (at 45.72 101.6 90))
     (property "Value" "?" (id 1) (at 48.26 101.6 90))
-    (property "Footprint" "" (id 2) (at 43.18 101.6 0)
+    (property "Footprint" "Capacitor_SMD:C_0805_2012Metric_Pad1.18x1.45mm_HandSolder" (id 2) (at 43.18 101.6 0)
       (effects (font (size 1.27 1.27)) hide)
     )
@@
     (property "Reference" "C9" (id 0) (at 63.5 83.82 90))
     (property "Value" "220n" (id 1) (at 66.04 83.82 90))
-    (property "Footprint" "" (id 2) (at 68.58 83.82 0)
+    (property "Footprint" "Capacitor_SMD:C_0805_2012Metric_Pad1.18x1.45mm_HandSolder" (id 2) (at 68.58 83.82 0)
       (effects (font (size 1.27 1.27)) hide)
     )
@@
       (effects (font (size 1.27 1.27)) (justify left))
     )
-    (property "Footprint" "" (id 2) (at 86.36 152.4 0)
+    (property "Footprint" "Capacitor_SMD:C_1206_3216Metric_Pad1.33x1.80mm_HandSolder" (id 2) (at 86.36 152.4 0)
       (effects (font (size 1.27 1.27)) hide)
     )
@@
     (in_bom yes) (on_board yes) (fields_autoplaced)
     (property "Reference" "L1" (id 0) (at 40.64 77.47 90))
-    (property "Value" "" (id 1) (at 40.64 80.01 90))
-    (property "Footprint" "" (id 2) (at 40.64 83.82 0)
+    (property "Value" "10u" (id 1) (at 40.64 80.01 90))
+    (property "Footprint" "Inductor_SMD:L_Taiyo-Yuden_MD-3030" (id 2) (at 40.64 83.82 0)
       (effects (font (size 1.27 1.27)) hide)
     )
@@
     (property "Reference" "U3" (id 0) (at 213.36 30.48 0))
     (property "Value" "RC4558" (id 1) (at 213.36 33.02 0))
-    (property "Footprint" "" (id 2) (at 213.36 40.64 0)
+    (property "Footprint" "Package_SO:SOIC-8-1EP_3.9x4.9mm_P1.27mm_EP2.514x3.2mm" (id 2) (at 213.36 40.64 0)
       (effects (font (size 1.27 1.27)) hide)
     )
@@
     (property "Reference" "C8" (id 0) (at 68.58 68.58 90))
     (property "Value" "1n" (id 1) (at 71.12 68.58 90))
-    (property "Footprint" "" (id 2) (at 66.04 68.58 0)
+    (property "Footprint" "Capacitor_SMD:C_0805_2012Metric_Pad1.18x1.45mm_HandSolder" (id 2) (at 66.04 68.58 0)
       (effects (font (size 1.27 1.27)) hide)
     )
@@
     (property "Reference" "R3" (id 0) (at 109.22 67.31 90))
     (property "Value" "34k" (id 1) (at 109.22 69.85 90))
-    (property "Footprint" "" (id 2) (at 109.22 73.66 0)
+    (property "Footprint" "Capacitor_SMD:C_0805_2012Metric_Pad1.18x1.45mm_HandSolder" (id 2) (at 109.22 73.66 0)
       (effects (font (size 1.27 1.27)) hide)
     )
@@
       (effects (font (size 1.27 1.27)) (justify right))
     )
-    (property "Value" "" (id 1) (at 30.48 88.9 90)
+    (property "Value" "PMEG100T10ELXD" (id 1) (at 30.48 88.9 90)
       (effects (font (size 1.27 1.27)) (justify right))
     )
-    (property "Footprint" "" (id 2) (at 55.245 88.9 0)
+    (property "Footprint" "Diode_SMD:D_SOD-323F" (id 2) (at 55.245 88.9 0)
       (effects (font (size 1.27 1.27)) hide)
     )
@@
       (effects (font (size 1.27 1.27)) (justify left))
     )
-    (property "Footprint" "" (id 2) (at 101.6 152.4 0)
+    (property "Footprint" "Capacitor_SMD:C_1206_3216Metric_Pad1.33x1.80mm_HandSolder" (id 2) (at 101.6 152.4 0)
       (effects (font (size 1.27 1.27)) hide)
     )
@@
       (effects (font (size 1.27 1.27)) (justify left))
     )
-    (property "Footprint" "" (id 2) (at 228.6 43.18 0)
+    (property "Footprint" "Capacitor_SMD:C_0805_2012Metric_Pad1.18x1.45mm_HandSolder" (id 2) (at 228.6 43.18 0)
       (effects (font (size 1.27 1.27)) hide)
     )
@@
       (effects (font (size 1.27 1.27)) (justify left))
     )
-    (property "Footprint" "" (id 2) (at 243.84 38.1 0)
+    (property "Footprint" "Capacitor_SMD:C_0805_2012Metric_Pad1.18x1.45mm_HandSolder" (id 2) (at 243.84 38.1 0)
       (effects (font (size 1.27 1.27)) hide)
     )
@@
     (in_bom yes) (on_board yes)
     (property "Reference" "C18" (id 0) (at 147.32 101.6 90))
-    (property "Value" "" (id 1) (at 149.86 101.6 90))
-    (property "Footprint" "" (id 2) (at 144.78 101.6 0)
+    (property "Value" "470n" (id 1) (at 149.86 101.6 90))
+    (property "Footprint" "Capacitor_SMD:C_0805_2012Metric_Pad1.18x1.45mm_HandSolder" (id 2) (at 144.78 101.6 0)
       (effects (font (size 1.27 1.27)) hide)
     )
@@
       (effects (font (size 1.27 1.27)) (justify left))
     )
-    (property "Footprint" "" (id 2) (at 111.76 152.4 0)
-      (effects (font (size 1.27 1.27)) hide)
-    )
+    (property "Footprint" "Capacitor_SMD:C_1206_3216Metric_Pad1.33x1.80mm_HandSolder" (id 2) (at 111.76 152.4 0)
+      (effects (font (size 1.27 1.27)) hide)
+    )
