File: hardware/power.kicad_sch (KiCad schematic)
At the start: 28 parts, among them U2 LT3988, U3 RC4558

Commit message: small changes
Parts:
- C10, C11, C13, C15, C7: footprint (none) -> Capacitor_SMD:C_1206_3216Metric_Pad1.33x1.80mm_HandSolder
- C12, C14, C16, C17, C19, C5, C8, C9, R1, R2, R3, R4, R5, R6, R7: footprint (none) -> Capacitor_SMD:C_0805_2012Metric_Pad1.18x1.45mm_HandSolder
- C18: value (none) -> 470n; footprint (none) -> Capacitor_SMD:C_0805_2012Metric_Pad1.18x1.45mm_HandSolder
- C6: value (none) -> 4.7u; footprint (none) -> Capacitor_SMD:C_1206_3216Metric_Pad1.33x1.80mm_HandSolder
- D1, D2: value (none) -> PMEG100T10ELXD; footprint (none) -> Diode_SMD:D_SOD-323F
- L1, L2: value (none) -> 10u; footprint (none) -> Inductor_SMD:L_Taiyo-Yuden_MD-3030
- U3: footprint (none) -> Package_SO:SOIC-8-1EP_3.9x4.9mm_P1.27mm_EP2.514x3.2mm
Other:
- note added: "physically partition grounds"
Changed lines of the file:
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@@
+    (effects (font (size 1.27 1.27)) (justify left bottom))
+  )
+  (text "physically partition grounds	" (at 101.6 116.84 0)
     (effects (font (size 1.27 1.27)) (justify left bottom))
   )
@@
     (property "Reference" "R5" (id 0) (at 119.38 90.17 90))
     (property "Value" "34k" (id 1) (at 119.38 92.71 90))
-    (property "Footprint" "" (id 2) (at 119.38 96.52 0)
+    (property "Footprint" "Capacitor_SMD:C_0805_2012Metric_Pad1.18x1.45mm_HandSolder" (id 2) (at 119.38 96.52 0)
       (effects (font (size 1.27 1.27)) hide)
     )
@@
       (effects (font (size 1.27 1.27)) (justify left))
     )
-    (property "Value" "" (id 1) (at 127 91.44 90)
-      (effects (font (size 1.27 1.27)) (justify left))
-    )
-    (property "Footprint" "" (id 2) (at 122.555 88.9 0)
+    (property "Value" "PMEG100T10ELXD" (id 1) (at 127 91.44 90)
+      (effects (font (size 1.27 1.27)) (justify left))
+    )
+    (property "Footprint" "Diode_SMD:D_SOD-323F" (id 2) (at 122.555 88.9 0)
       (effects (font (size 1.27 1.27)) hide)
     )
@@
     (property "Reference" "C17" (id 0) (at 119.38 104.14 90))
     (property "Value" "22p" (id 1) (at 119.38 106.68 90))
-    (property "Footprint" "" (id 2) (at 119.38 101.6 0)
+    (property "Footprint" "Capacitor_SMD:C_0805_2012Metric_Pad1.18x1.45mm_HandSolder" (id 2) (at 119.38 101.6 0)
       (effects (font (size 1.27 1.27)) hide)
     )
@@
       (effects (font (size 1.27 1.27)) (justify left))
     )
-    (property "Footprint" "" (id 2) (at 256.54 38.1 0)
+    (property "Footprint" "Package_SO:SOIC-8-1EP_3.9x4.9mm_P1.27mm_EP2.514x3.2mm" (id 2) (at 256.54 38.1 0)
       (effects (font (size 1.27 1.27)) hide)
     )
@@
       (effects (font (size 1.27 1.27)) (justify left))
     )
-    (property "Footprint" "" (id 2) (at 228.6 33.02 0)
+    (property "Footprint" "Capacitor_SMD:C_0805_2012Metric_Pad1.18x1.45mm_HandSolder" (id 2) (at 228.6 33.02 0)
       (effects (font (size 1.27 1.27)) hide)
     )
@@
     (property "Reference" "C16" (id 0) (at 116.84 68.58 90))
     (property "Value" "1n" (id 1) (at 119.38 68.58 90))
-    (property "Footprint" "" (id 2) (at 114.3 68.58 0)
+    (property "Footprint" "Capacitor_SMD:C_0805_2012Metric_Pad1.18x1.45mm_HandSolder" (id 2) (at 114.3 68.58 0)
       (effects (font (size 1.27 1.27)) hide)
     )
@@
     (in_bom yes) (on_board yes) (fields_autoplaced)
     (property "Reference" "L2" (id 0) (at 134.62 77.47 90))
-    (property "Value" "" (id 1) (at 134.62 80.01 90))
-    (property "Footprint" "" (id 2) (at 134.62 83.82 0)
+    (property "Value" "10u" (id 1) (at 134.62 80.01 90))
+    (property "Footprint" "Inductor_SMD:L_Taiyo-Yuden_MD-3030" (id 2) (at 134.62 83.82 0)
       (effects (font (size 1.27 1.27)) hide)
     )
@@
       (effects (font (size 1.27 1.27)) (justify right))
     )
-    (property "Footprint" "" (id 2) (at 109.22 104.14 0)
+    (property "Footprint" "Capacitor_SMD:C_0805_2012Metric_Pad1.18x1.45mm_HandSolder" (id 2) (at 109.22 104.14 0)
       (effects (font (size 1.27 1.27)) hide)
     )
@@
     (property "Reference" "R1" (id 0) (at 60.96 90.17 90))
     (property "Value" "150k" (id 1) (at 60.96 92.71 90))
-    (property "Footprint" "" (id 2) (at 60.96 96.52 0)
+    (property "Footprint" "Capacitor_SMD:C_0805_2012Metric_Pad1.18x1.45mm_HandSolder" (id 2) (at 60.96 96.52 0)
       (effects (font (size 1.27 1.27)) hide)
     )
@@
     (property "Reference" "C12" (id 0) (at 99.06 45.72 90))
     (property "Value" "22p" (id 1) (at 101.6 45.72 90))
-    (property "Footprint" "" (id 2) (at 96.52 45.72 0)
+    (property "Footprint" "Capacitor_SMD:C_0805_2012Metric_Pad1.18x1.45mm_HandSolder" (id 2) (at 96.52 45.72 0)
       (effects (font (size 1.27 1.27)) hide)
     )
@@
       (effects (font (size 1.27 1.27)) (justify left))
     )
-    (property "Value" "" (id 1) (at 53.34 153.6762 0)
-      (effects (font (size 1.27 1.27)) (justify left))
-    )
-    (property "Footprint" "" (id 2) (at 50.8 152.4 0)
+    (property "Value" "4.7u" (id 1) (at 53.34 153.6762 0)
+      (effects (font (size 1.27 1.27)) (justify left))
+    )
+    (property "Footprint" "Capacitor_SMD:C_1206_3216Metric_Pad1.33x1.80mm_HandSolder" (id 2) (at 50.8 152.4 0)
       (effects (font (size 1.27 1.27)) hide)
     )
@@
     (property "Reference" "C14" (id 0) (at 111.76 83.82 90))
     (property "Value" "220n" (id 1) (at 114.3 83.82 90))
-    (property "Footprint" "" (id 2) (at 109.22 83.82 0)
+    (property "Footprint" "Capacitor_SMD:C_0805_2012Metric_Pad1.18x1.45mm_HandSolder" (id 2) (at 109.22 83.82 0)
       (effects (font (size 1.27 1.27)) hide)
     )
@@
       (effects (font (size 1.27 1.27)) (justify left))
     )
-    (property "Footprint" "" (id 2) (at 76.2 152.4 0)
+    (property "Footprint" "Capacitor_SMD:C_1206_3216Metric_Pad1.33x1.80mm_HandSolder" (id 2) (at 76.2 152.4 0)
       (effects (font (size 1.27 1.27)) hide)
     )
@@
       (effects (font (size 1.27 1.27)) (justify right))
     )
-    (property "Footprint" "" (id 2) (at 68.58 104.14 0)
+    (property "Footprint" "Capacitor_SMD:C_0805_2012Metric_Pad1.18x1.45mm_HandSolder" (id 2) (at 68.58 104.14 0)
       (effects (font (size 1.27 1.27)) hide)
     )
@@
       (effects (font (size 1.27 1.27)) (justify left))
     )
-    (property "Footprint" "" (id 2) (at 60.96 152.4 0)
+    (property "Footprint" "Capacitor_SMD:C_1206_3216Metric_Pad1.33x1.80mm_HandSolder" (id 2) (at 60.96 152.4 0)
       (effects (font (size 1.27 1.27)) hide)
     )
@@
     (property "Reference" "C5" (id 0) (at 45.72 101.6 90))
     (property "Value" "?" (id 1) (at 48.26 101.6 90))
-    (property "Footprint" "" (id 2) (at 43.18 101.6 0)
+    (property "Footprint" "Capacitor_SMD:C_0805_2012Metric_Pad1.18x1.45mm_HandSolder" (id 2) (at 43.18 101.6 0)
       (effects (font (size 1.27 1.27)) hide)
     )
@@
     (property "Reference" "C9" (id 0) (at 63.5 83.82 90))
     (property "Value" "220n" (id 1) (at 66.04 83.82 90))
-    (property "Footprint" "" (id 2) (at 68.58 83.82 0)
+    (property "Footprint" "Capacitor_SMD:C_0805_2012Metric_Pad1.18x1.45mm_HandSolder" (id 2) (at 68.58 83.82 0)
       (effects (font (size 1.27 1.27)) hide)
     )
@@
       (effects (font (size 1.27 1.27)) (justify left))
     )
-    (property "Footprint" "" (id 2) (at 86.36 152.4 0)
+    (property "Footprint" "Capacitor_SMD:C_1206_3216Metric_Pad1.33x1.80mm_HandSolder" (id 2) (at 86.36 152.4 0)
       (effects (font (size 1.27 1.27)) hide)
     )
@@
     (in_bom yes) (on_board yes) (fields_autoplaced)
     (property "Reference" "L1" (id 0) (at 40.64 77.47 90))
-    (property "Value" "" (id 1) (at 40.64 80.01 90))
-    (property "Footprint" "" (id 2) (at 40.64 83.82 0)
+    (property "Value" "10u" (id 1) (at 40.64 80.01 90))
+    (property "Footprint" "Inductor_SMD:L_Taiyo-Yuden_MD-3030" (id 2) (at 40.64 83.82 0)
       (effects (font (size 1.27 1.27)) hide)
     )
@@
     (property "Reference" "U3" (id 0) (at 213.36 30.48 0))
     (property "Value" "RC4558" (id 1) (at 213.36 33.02 0))
-    (property "Footprint" "" (id 2) (at 213.36 40.64 0)
+    (property "Footprint" "Package_SO:SOIC-8-1EP_3.9x4.9mm_P1.27mm_EP2.514x3.2mm" (id 2) (at 213.36 40.64 0)
       (effects (font (size 1.27 1.27)) hide)
     )
@@
     (property "Reference" "C8" (id 0) (at 68.58 68.58 90))
     (property "Value" "1n" (id 1) (at 71.12 68.58 90))
-    (property "Footprint" "" (id 2) (at 66.04 68.58 0)
+    (property "Footprint" "Capacitor_SMD:C_0805_2012Metric_Pad1.18x1.45mm_HandSolder" (id 2) (at 66.04 68.58 0)
       (effects (font (size 1.27 1.27)) hide)
     )
@@
     (property "Reference" "R3" (id 0) (at 109.22 67.31 90))
     (property "Value" "34k" (id 1) (at 109.22 69.85 90))
-    (property "Footprint" "" (id 2) (at 109.22 73.66 0)
+    (property "Footprint" "Capacitor_SMD:C_0805_2012Metric_Pad1.18x1.45mm_HandSolder" (id 2) (at 109.22 73.66 0)
       (effects (font (size 1.27 1.27)) hide)
     )
@@
       (effects (font (size 1.27 1.27)) (justify right))
     )
-    (property "Value" "" (id 1) (at 30.48 88.9 90)
+    (property "Value" "PMEG100T10ELXD" (id 1) (at 30.48 88.9 90)
       (effects (font (size 1.27 1.27)) (justify right))
     )
-    (property "Footprint" "" (id 2) (at 55.245 88.9 0)
+    (property "Footprint" "Diode_SMD:D_SOD-323F" (id 2) (at 55.245 88.9 0)
       (effects (font (size 1.27 1.27)) hide)
     )
@@
       (effects (font (size 1.27 1.27)) (justify left))
     )
-    (property "Footprint" "" (id 2) (at 101.6 152.4 0)
+    (property "Footprint" "Capacitor_SMD:C_1206_3216Metric_Pad1.33x1.80mm_HandSolder" (id 2) (at 101.6 152.4 0)
       (effects (font (size 1.27 1.27)) hide)
     )
@@
       (effects (font (size 1.27 1.27)) (justify left))
     )
-    (property "Footprint" "" (id 2) (at 228.6 43.18 0)
+    (property "Footprint" "Capacitor_SMD:C_0805_2012Metric_Pad1.18x1.45mm_HandSolder" (id 2) (at 228.6 43.18 0)
       (effects (font (size 1.27 1.27)) hide)
     )
@@
       (effects (font (size 1.27 1.27)) (justify left))
     )
-    (property "Footprint" "" (id 2) (at 243.84 38.1 0)
+    (property "Footprint" "Capacitor_SMD:C_0805_2012Metric_Pad1.18x1.45mm_HandSolder" (id 2) (at 243.84 38.1 0)
       (effects (font (size 1.27 1.27)) hide)
     )
@@
     (in_bom yes) (on_board yes)
     (property "Reference" "C18" (id 0) (at 147.32 101.6 90))
-    (property "Value" "" (id 1) (at 149.86 101.6 90))
-    (property "Footprint" "" (id 2) (at 144.78 101.6 0)
+    (property "Value" "470n" (id 1) (at 149.86 101.6 90))
+    (property "Footprint" "Capacitor_SMD:C_0805_2012Metric_Pad1.18x1.45mm_HandSolder" (id 2) (at 144.78 101.6 0)
       (effects (font (size 1.27 1.27)) hide)
     )
@@
       (effects (font (size 1.27 1.27)) (justify left))
     )
-    (property "Footprint" "" (id 2) (at 111.76 152.4 0)
-      (effects (font (size 1.27 1.27)) hide)
-    )
+    (property "Footprint" "Capacitor_SMD:C_1206_3216Metric_Pad1.33x1.80mm_HandSolder" (id 2) (at 111.76 152.4 0)
+      (effects (font (size 1.27 1.27)) hide)
+    )

Commit message: microcontroller done?
Parts:
- removed C12, C17: 22p, Capacitor_SMD:C_0805_2012Metric_Pad1.18x1.45mm_HandSolder, symbol Device:C_Small
- removed C19: 100n, Capacitor_SMD:C_0805_2012Metric_Pad1.18x1.45mm_HandSolder, symbol Device:C_Small
- removed C5: ?, Capacitor_SMD:C_0805_2012Metric_Pad1.18x1.45mm_HandSolder, symbol Device:C_Small
- removed R2, R4, R7: 10k, Capacitor_SMD:C_0805_2012Metric_Pad1.18x1.45mm_HandSolder, symbol Device:R_Small_US
- added C? (x2): 22p, Capacitor_SMD:C_0402_1005Metric_Pad0.74x0.62mm_HandSolder, symbol Device:C
- added C?: 470n, Capacitor_SMD:C_0805_2012Metric_Pad1.18x1.45mm_HandSolder, symbol Device:C_Small
- added C?: 100n, Capacitor_SMD:C_0402_1005Metric, symbol Device:C
- added R? (x3): 10k, Resistor_SMD:R_0805_2012Metric, symbol Device:R_Small_US
- R9: renamed from R6; footprint Capacitor_SMD:C_0805_2012Metric_Pad1.18x1.45mm_HandSolder -> Resistor_SMD:R_0805_2012Metric; Mouser (none) -> https://www.mouser.com/ProductDetail/Panasonic/ERJ-6ENF1002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
- renumbered C8 to C10, C9 to C11, C10 to C12, C11 to C13, C13 to C15, C14 to C16, C15 to C17, C16 to C18, C18 to C20, C6 to C8, C7 to C9, R1 to R4, R3 to R6, R5 to R8
Connections:
- net +3V3: now also C?.1, C?.2
- net GND: now also C?.1, R?.2; no longer C10.1, C12.2, C13.2, C15.2, C17.2, C18.1, C20.1, C8.2, C9.2, R6.2, U2.12 (SYNC), U2.17 (GND)
- net VCC: now also C?.2
- net VDD: now also C?.2
- net at R8.2, U2.11 (FB2): now also C?.2, R?.1
- net at R9.2, U3.3 (+): now also R?.1
- net at R4.1, U2.14 (FB1): now also R?.1
- new net GNDPWR: C10.1, C12.2, C13.2, C15.2, C17.2, C18.1, C20.1, C8.2, C9.2, C?.1, C?.1, R6.2, R?.2, R?.2, U2.12 (SYNC), U2.17 (GND)
Other:
- note removed: "physically partition grounds"

Commit message: sourcing parts
Parts:
- removed C10: 1n, Capacitor_SMD:C_0805_2012Metric_Pad1.18x1.45mm_HandSolder, symbol Device:C_Small
- removed C11: 220n, Capacitor_SMD:C_0805_2012Metric_Pad1.18x1.45mm_HandSolder, symbol Device:C_Small
- removed C?: 470n, Capacitor_SMD:C_0805_2012Metric_Pad1.18x1.45mm_HandSolder, symbol Device:C_Small
- removed R6, R8: 34k, Capacitor_SMD:C_0805_2012Metric_Pad1.18x1.45mm_HandSolder, symbol Device:R_Small_US
- added C?: 470n, Capacitor_SMD:C_0805_2012Metric_Pad1.18x1.45mm_HandSolder, symbol Device:C_Small
- added C?: 220n, Capacitor_SMD:C_0805_2012Metric_Pad1.18x1.45mm_HandSolder, symbol Device:C_Small
- added C?: 1n, Capacitor_SMD:C_0805_2012Metric_Pad1.18x1.45mm_HandSolder, symbol Device:C_Small
- added R? (x2): 34k, Resistor_SMD:R_0805_2012Metric, symbol Device:R_Small_US
- C16, C18, C20: Mouser (none) -> https://www.mouser.com/ProductDetail/Murata-Electronics/GRM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
- R4: footprint Capacitor_SMD:C_0805_2012Metric_Pad1.18x1.45mm_HandSolder -> Resistor_SMD:R_0805_2012Metric; Mouser (none) -> https://www.mouser.com/ProductDetail/Panasonic/ERJ-U06F1503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
Connections:
- net +3V3: now also R?.1
- net GNDPWR: now also C?.1, C?.1, R?.1
- net at C?.2, R?.1, U2.11 (FB2): now also R?.2
- net at U2.3 (BOOST1): now also C?.2
- net at D1.1 (K), L1.2, U2.2 (SW1): now also C?.1
- net at U2.13 (RT): now also R?.2
- net at U2.15 (TRACK/SS1): now also C?.2
- net VCC renamed VS
- net VDD renamed +12V
- net +12V: now also C?.2

Commit message: swd interface
Parts:
- R4: footprint Resistor_SMD:R_0805_2012Metric -> Capacitor_SMD:C_0805_2012Metric_Pad1.18x1.45mm_HandSolder
- gave numbers to parts that had none: 11
Changed lines of the file:
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@@
   (symbol (lib_id "Device:C") (at 96.52 45.72 180) (unit 1)
     (in_bom yes) (on_board yes) (fields_autoplaced)
-    (property "Reference" "C?" (id 0) (at 100.33 44.4499 0)
+    (property "Reference" "C14" (id 0) (at 100.33 44.4499 0)
       (effects (font (size 1.27 1.27)) (justify right))
     )
@@
   (symbol (lib_id "power:GNDPWR") (at 96.52 49.53 0) (unit 1)
     (in_bom yes) (on_board yes) (fields_autoplaced)
-    (property "Reference" "#PWR?" (id 0) (at 96.52 54.61 0)
+    (property "Reference" "#PWR015" (id 0) (at 96.52 54.61 0)
       (effects (font (size 1.27 1.27)) hide)
     )
@@
   (symbol (lib_id "power:+12V") (at 27.94 81.28 0) (unit 1)
     (in_bom yes) (on_board yes) (fields_autoplaced)
-    (property "Reference" "#PWR?" (id 0) (at 27.94 85.09 0)
+    (property "Reference" "#PWR09" (id 0) (at 27.94 85.09 0)
       (effects (font (size 1.27 1.27)) hide)
     )
@@
   (symbol (lib_id "power:VS") (at 91.44 38.1 0) (unit 1)
     (in_bom yes) (on_board yes) (fields_autoplaced)
-    (property "Reference" "#PWR?" (id 0) (at 86.36 41.91 0)
+    (property "Reference" "#PWR014" (id 0) (at 86.36 41.91 0)
       (effects (font (size 1.27 1.27)) hide)
     )
@@
   (symbol (lib_id "Device:C_Small") (at 43.18 101.6 180) (unit 1)
     (in_bom yes) (on_board yes)
-    (property "Reference" "C?" (id 0) (at 45.72 101.6 90))
+    (property "Reference" "C7" (id 0) (at 45.72 101.6 90))
     (property "Value" "470n" (id 1) (at 48.26 101.6 90))
     (property "Footprint" "Capacitor_SMD:C_0805_2012Metric_Pad1.18x1.45mm_HandSolder" (id 2) (at 43.18 101.6 0)
@@
   (symbol (lib_id "Device:C") (at 119.38 101.6 270) (mirror x) (unit 1)
     (in_bom yes) (on_board yes)
-    (property "Reference" "C?" (id 0) (at 123.19 106.68 90))
+    (property "Reference" "C19" (id 0) (at 123.19 106.68 90))
     (property "Value" "22p" (id 1) (at 123.19 104.14 90))
     (property "Footprint" "Capacitor_SMD:C_0402_1005Metric_Pad0.74x0.62mm_HandSolder" (id 2) (at 115.57 100.6348 0)
@@
     (property "Reference" "R4" (id 0) (at 60.96 90.17 90))
     (property "Value" "150k" (id 1) (at 60.96 92.71 90))
-    (property "Footprint" "Resistor_SMD:R_0805_2012Metric" (id 2) (at 60.96 96.52 0)
+    (property "Footprint" "Capacitor_SMD:C_0805_2012Metric_Pad1.18x1.45mm_HandSolder" (id 2) (at 60.96 96.52 0)
       (effects (font (size 1.27 1.27)) hide)
     )
@@
   (symbol (lib_id "Device:R_Small_US") (at 68.58 104.14 0) (unit 1)
     (in_bom yes) (on_board yes) (fields_autoplaced)
-    (property "Reference" "R?" (id 0) (at 71.12 102.8699 0)
+    (property "Reference" "R5" (id 0) (at 71.12 102.8699 0)
       (effects (font (size 1.27 1.27)) (justify left))
     )
@@
   (symbol (lib_id "Device:C_Small") (at 68.58 83.82 180) (unit 1)
     (in_bom yes) (on_board yes)
-    (property "Reference" "C?" (id 0) (at 71.12 83.82 90))
+    (property "Reference" "C11" (id 0) (at 71.12 83.82 90))
     (property "Value" "220n" (id 1) (at 73.66 83.82 90))
     (property "Footprint" "Capacitor_SMD:C_0805_2012Metric_Pad1.18x1.45mm_HandSolder" (id 2) (at 68.58 83.82 0)
@@
   (symbol (lib_id "Device:R_Small_US") (at 109.22 104.14 0) (unit 1)
     (in_bom yes) (on_board yes) (fields_autoplaced)
-    (property "Reference" "R?" (id 0) (at 111.76 102.8699 0)
+    (property "Reference" "R7" (id 0) (at 111.76 102.8699 0)
       (effects (font (size 1.27 1.27)) (justify left))
     )
@@
   (symbol (lib_id "Device:R_Small_US") (at 119.38 96.52 270) (unit 1)
     (in_bom yes) (on_board yes) (fields_autoplaced)
-    (property "Reference" "R?" (id 0) (at 119.38 90.17 90))
+    (property "Reference" "R8" (id 0) (at 119.38 90.17 90))
     (property "Value" "34k" (id 1) (at 119.38 92.71 90))
     (property "Footprint" "Resistor_SMD:R_0805_2012Metric" (id 2) (at 119.38 96.52 0)
@@
   (symbol (lib_id "Device:C") (at 243.84 38.1 0) (mirror x) (unit 1)
     (in_bom yes) (on_board yes) (fields_autoplaced)
-    (property "Reference" "C?" (id 0) (at 240.03 36.8299 0)
+    (property "Reference" "C21" (id 0) (at 240.03 36.8299 0)
       (effects (font (size 1.27 1.27)) (justify right))
     )
@@
   (symbol (lib_id "Device:R_Small_US") (at 109.22 73.66 270) (unit 1)
     (in_bom yes) (on_board yes) (fields_autoplaced)
-    (property "Reference" "R?" (id 0) (at 109.22 67.31 90))
+    (property "Reference" "R6" (id 0) (at 109.22 67.31 90))
     (property "Value" "34k" (id 1) (at 109.22 69.85 90))
     (property "Footprint" "Resistor_SMD:R_0805_2012Metric" (id 2) (at 109.22 73.66 0)
@@
   (symbol (lib_id "Device:R_Small_US") (at 228.6 43.18 0) (unit 1)
     (in_bom yes) (on_board yes) (fields_autoplaced)
-    (property "Reference" "R?" (id 0) (at 231.14 41.9099 0)
+    (property "Reference" "R10" (id 0) (at 231.14 41.9099 0)
       (effects (font (size 1.27 1.27)) (justify left))
     )
@@
   (symbol (lib_id "Device:C_Small") (at 66.04 68.58 180) (unit 1)
     (in_bom yes) (on_board yes)
-    (property "Reference" "C?" (id 0) (at 68.58 68.58 90))
+    (property "Reference" "C10" (id 0) (at 68.58 68.58 90))
     (property "Value" "1n" (id 1) (at 71.12 68.58 90))
     (property "Footprint" "Capacitor_SMD:C_0805_2012Metric_Pad1.18x1.45mm_HandSolder" (id 2) (at 66.04 68.58 0)
@@
   (symbol (lib_id "power:GNDPWR") (at 50.8 165.1 0) (unit 1)
     (in_bom yes) (on_board yes) (fields_autoplaced)
-    (property "Reference" "#PWR?" (id 0) (at 50.8 170.18 0)
+    (property "Reference" "#PWR011" (id 0) (at 50.8 170.18 0)
       (effects (font (size 1.27 1.27)) hide)
     )
@@
   (symbol (lib_id "power:GNDPWR") (at 114.3 73.66 0) (unit 1)
     (in_bom yes) (on_board yes)
-    (property "Reference" "#PWR?" (id 0) (at 114.3 78.74 0)
+    (property "Reference" "#PWR016" (id 0) (at 114.3 78.74 0)
       (effects (font (size 1.27 1.27)) hide)
     )
@@
   (symbol (lib_id "power:GNDPWR") (at 88.9 111.76 0) (unit 1)
     (in_bom yes) (on_board yes) (fields_autoplaced)
-    (property "Reference" "#PWR?" (id 0) (at 88.9 116.84 0)
+    (property "Reference" "#PWR013" (id 0) (at 88.9 116.84 0)
       (effects (font (size 1.27 1.27)) hide)
     )
@@
   (symbol (lib_id "power:GNDPWR") (at 66.04 73.66 0) (unit 1)
     (in_bom yes) (on_board yes) (fields_autoplaced)
-    (property "Reference" "#PWR?" (id 0) (at 66.04 78.74 0)
+    (property "Reference" "#PWR012" (id 0) (at 66.04 78.74 0)
       (effects (font (size 1.27 1.27)) hide)
     )
@@
   (symbol (lib_id "power:VS") (at 50.8 139.7 0) (unit 1)
     (in_bom yes) (on_board yes) (fields_autoplaced)
-    (property "Reference" "#PWR?" (id 0) (at 45.72 143.51 0)
-      (effects (font (size 1.27 1.27)) hide)
-    )
+    (property "Reference" "#PWR010" (id 0) (at 45.72 143.51 0)
+      (effects (font (size 1.27 1.27)) hide)
+    )
