File: hardware/driver.kicad_sch (KiCad schematic)
At the start: 0 parts

Commit message: Version 1 of driver and current sense.
Parts:
- added C? (x9): 100n, symbol Device:C_Small
- added R? (x2): 2m, symbol Device:R_Small_US
- added R? (x3): 10, symbol Device:R_Small_US
- added R?: (no value), symbol Device:R_Small_US
- added U? (x3): INA181A2IDBVT, symbol INA181A2IDBVT:INA181A2IDBVT
- added U? (x3): EPC2152, symbol EPC2152:EPC2152
Connections:
- new net: C?.1, R?.1, U?.3 (IN+), U?.6 (SW) (x3)
- new net: R?.2, U?.4 (IN-) (x3)
- new net: C?.2, R?.1 (x3)
- new net: R?.2, U?.1 (Vboot) (x3)
- new net +3V3: C?.1, C?.1, C?.1, U?.6 (VS), U?.6 (VS), U?.6 (VS)
- new net GND: C?.2, C?.2, C?.2, C?.2, C?.2, C?.2, U?.2 (GND), U?.2 (GND), U?.2 (GND), U?.7 (GND), U?.7 (GND), U?.7 (GND)
- new net ISNS_A: U?.1 (OUT)
- new net ISNS_B: U?.1 (OUT)
- new net ISNS_C: U?.1 (OUT)
- new net PWM_AB: U?.4 (LSin)
- new net PWM_AT: U?.3 (HSin)
- new net PWM_BB: U?.4 (LSin)
- new net PWM_BT: U?.3 (HSin)
- new net PWM_CB: U?.4 (LSin)
- new net PWM_CT: U?.3 (HSin)
- new net VCC: U?.5 (VIN), U?.5 (VIN), U?.5 (VIN)
- new net VDD: C?.1, C?.1, C?.1, U?.2 (Vdd), U?.2 (Vdd), U?.2 (Vdd)
Other:
- note added: "Rboost to be investigated later."
- note added: "ravi to-do: calculate and add bulk capacitance add voltage measurement circuit add buck regulator do we need/want filtering on current sense?"
- note added: "res: WSKW06122L000FEA 0612 package"

Commit message: added buck converter rev1
still need to pick inductors, size bulk capacitance, verify calcs
Parts:
- R?: value (none) -> 2m
Connections:
- net PH_C: now reaches R?.2, U?.4 (IN-)
- net PH_B: now reaches R?.2, U?.4 (IN-)
- net PH_A: now reaches R?.2, U?.4 (IN-)
Changed lines of the file:
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@@
 (kicad_sch (version 20211123) (generator eeschema)
   (paper "A4")
+  (junction (at 101.6 99.06) (diameter 0) (color 0 0 0 0)
+  )
   (junction (at 137.16 25.4) (diameter 0) (color 0 0 0 0)
   )
@@
   (junction (at 35.56 25.4) (diameter 0) (color 0 0 0 0)
   )
+  (junction (at 203.2 43.18) (diameter 0) (color 0 0 0 0)
+  )
   (junction (at 175.26 43.18) (diameter 0) (color 0 0 0 0)
   )
@@
   (junction (at 35.56 81.28) (diameter 0) (color 0 0 0 0)
   )
+  (junction (at 101.6 43.18) (diameter 0) (color 0 0 0 0)
+  )
   (junction (at 73.66 99.06) (diameter 0) (color 0 0 0 0)
   )
@@
     (stroke (width 0) (type default) (color 0 0 0 0))
   )
+  (wire (pts (xy 203.2 43.18) (xy 205.74 43.18))
+    (stroke (width 0) (type default) (color 0 0 0 0))
+  )
   (wire (pts (xy 83.82 53.34) (xy 81.28 53.34))
     (stroke (width 0) (type default) (color 0 0 0 0))
@@
   )
   (wire (pts (xy 185.42 53.34) (xy 182.88 53.34))
+    (stroke (width 0) (type default) (color 0 0 0 0))
+  )
+  (wire (pts (xy 101.6 43.18) (xy 104.14 43.18))
+    (stroke (width 0) (type default) (color 0 0 0 0))
+  )
+  (wire (pts (xy 101.6 99.06) (xy 104.14 99.06))
     (stroke (width 0) (type default) (color 0 0 0 0))
   )
@@
     )
   )
+  (global_label "PH_C" (shape input) (at 104.14 99.06 0) (fields_autoplaced)
+    (effects (font (size 1.27 1.27)) (justify left))
+    (property "Intersheet References" "${INTERSHEET_REFS}" (id 0) (at 111.3912 98.9806 0)
+      (effects (font (size 1.27 1.27)) (justify left) hide)
+    )
+  )
   (global_label "PWM_BT" (shape input) (at 134.62 43.18 180) (fields_autoplaced)
     (effects (font (size 1.27 1.27)) (justify right))
@@
     )
   )
+  (global_label "PH_B" (shape input) (at 205.74 43.18 0) (fields_autoplaced)
+    (effects (font (size 1.27 1.27)) (justify left))
+    (property "Intersheet References" "${INTERSHEET_REFS}" (id 0) (at 212.9912 43.1006 0)
+      (effects (font (size 1.27 1.27)) (justify left) hide)
+    )
+  )
   (global_label "PWM_CT" (shape input) (at 33.02 99.06 180) (fields_autoplaced)
     (effects (font (size 1.27 1.27)) (justify right))
     (property "Intersheet References" "${INTERSHEET_REFS}" (id 0) (at 23.2288 98.9806 0)
       (effects (font (size 1.27 1.27)) (justify right) hide)
+    )
+  )
+  (global_label "PH_A" (shape input) (at 104.14 43.18 0) (fields_autoplaced)
+    (effects (font (size 1.27 1.27)) (justify left))
+    (property "Intersheet References" "${INTERSHEET_REFS}" (id 0) (at 111.2098 43.1006 0)
+      (effects (font (size 1.27 1.27)) (justify left) hide)
     )
   )
@@
     (in_bom yes) (on_board yes) (fields_autoplaced)
     (property "Reference" "R?" (id 0) (at 91.44 36.83 90))
-    (property "Value" "" (id 1) (at 91.44 39.37 90))
+    (property "Value" "2m" (id 1) (at 91.44 39.37 90))
     (property "Footprint" "" (id 2) (at 91.44 43.18 0)
       (effects (font (size 1.27 1.27)) hide)

Commit message: Started Buck Layout
Parts:
- removed R? (x2): 2m, symbol Device:R_Small_US
- added R11, R13: 2m, symbol Device:R_Small_US
- R10: renamed from R?; value 2m -> (none); Mouser (none) -> https://www.mouser.com/ProductDetail/Vishay-Dale/WSKW06122L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
- gave numbers to parts that had none: 18
Connections:
- net PH_B: now also R13.2
- net PH_C: now also R11.2
- net at C23.1, U5.6 (SW), U7.3 (IN+): now also R11.1
- net at C27.1, U8.6 (SW), U9.3 (IN+): now also R13.1
Other:
- note added: "ravi to-do: add voltage measurement circuit"
- note removed: "ravi to-do: calculate and add bulk capacitance add voltage measurement circuit add buck regulator do we need/want filtering on current sense?"

Commit message: small changes
Parts:
- C20, C21, C22, C23, C24, C25, C26, C27, C28, R12, R8, R9: footprint (none) -> Capacitor_SMD:C_0805_2012Metric_Pad1.18x1.45mm_HandSolder
- R10: value (none) -> 2m; footprint (none) -> SnapEDA Library:WSKW06122L000FEA
- R11, R13: footprint (none) -> SnapEDA Library:WSKW06122L000FEA
- U4, U5, U8: footprint (none) -> SnapEDA Library:EPC2152
- U6, U7, U9: footprint (none) -> Package_TO_SOT_SMD:SOT-23-6_Handsoldering
Changed lines of the file:
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@@
       (effects (font (size 1.27 1.27)) (justify left))
     )
-    (property "Footprint" "" (id 2) (at 127 30.48 0)
+    (property "Footprint" "Capacitor_SMD:C_0805_2012Metric_Pad1.18x1.45mm_HandSolder" (id 2) (at 127 30.48 0)
       (effects (font (size 1.27 1.27)) hide)
     )
@@
     (property "Reference" "U9" (id 0) (at 193.04 45.72 0))
     (property "Value" "INA181A2IDBVT" (id 1) (at 193.04 48.26 0))
-    (property "Footprint" "" (id 2) (at 193.04 63.5 0)
+    (property "Footprint" "Package_TO_SOT_SMD:SOT-23-6_Handsoldering" (id 2) (at 193.04 63.5 0)
       (effects (font (size 1.27 1.27)) hide)
     )
@@
     (property "Reference" "U7" (id 0) (at 91.44 101.6 0))
     (property "Value" "INA181A2IDBVT" (id 1) (at 91.44 104.14 0))
-    (property "Footprint" "" (id 2) (at 91.44 119.38 0)
+    (property "Footprint" "Package_TO_SOT_SMD:SOT-23-6_Handsoldering" (id 2) (at 91.44 119.38 0)
       (effects (font (size 1.27 1.27)) hide)
     )
@@
       (effects (font (size 1.27 1.27)) (justify left))
     )
-    (property "Footprint" "" (id 2) (at 147.32 33.02 0)
+    (property "Footprint" "Capacitor_SMD:C_0805_2012Metric_Pad1.18x1.45mm_HandSolder" (id 2) (at 147.32 33.02 0)
       (effects (font (size 1.27 1.27)) hide)
     )
@@
       (effects (font (size 1.27 1.27)) (justify left))
     )
-    (property "Footprint" "" (id 2) (at 45.72 81.28 0)
+    (property "Footprint" "Capacitor_SMD:C_0805_2012Metric_Pad1.18x1.45mm_HandSolder" (id 2) (at 45.72 81.28 0)
       (effects (font (size 1.27 1.27)) hide)
     )
@@
       (effects (font (size 1.27 1.27)) (justify left))
     )
-    (property "Footprint" "" (id 2) (at 45.72 25.4 0)
+    (property "Footprint" "Capacitor_SMD:C_0805_2012Metric_Pad1.18x1.45mm_HandSolder" (id 2) (at 45.72 25.4 0)
       (effects (font (size 1.27 1.27)) hide)
     )
@@
     (in_bom yes) (on_board yes) (fields_autoplaced)
     (property "Reference" "R10" (id 0) (at 91.44 36.83 90))
-    (property "Value" "" (id 1) (at 91.44 39.37 90))
-    (property "Footprint" "" (id 2) (at 91.44 43.18 0)
+    (property "Value" "2m" (id 1) (at 91.44 39.37 90))
+    (property "Footprint" "SnapEDA Library:WSKW06122L000FEA" (id 2) (at 91.44 43.18 0)
       (effects (font (size 1.27 1.27)) hide)
     )
@@
       (effects (font (size 1.27 1.27)) (justify left))
     )
-    (property "Footprint" "" (id 2) (at 25.4 30.48 0)
+    (property "Footprint" "Capacitor_SMD:C_0805_2012Metric_Pad1.18x1.45mm_HandSolder" (id 2) (at 25.4 30.48 0)
       (effects (font (size 1.27 1.27)) hide)
     )
@@
     (property "Reference" "U4" (id 0) (at 58.42 30.48 0))
     (property "Value" "EPC2152" (id 1) (at 58.42 33.02 0))
-    (property "Footprint" "" (id 2) (at 61.595 31.75 0)
+    (property "Footprint" "SnapEDA Library:EPC2152" (id 2) (at 61.595 31.75 0)
       (effects (font (size 1.27 1.27)) hide)
     )
@@
       (effects (font (size 1.27 1.27)) (justify left))
     )
-    (property "Footprint" "" (id 2) (at 25.4 86.36 0)
+    (property "Footprint" "Capacitor_SMD:C_0805_2012Metric_Pad1.18x1.45mm_HandSolder" (id 2) (at 25.4 86.36 0)
       (effects (font (size 1.27 1.27)) hide)
     )
@@
     (property "Reference" "R11" (id 0) (at 91.44 92.71 90))
     (property "Value" "2m" (id 1) (at 91.44 95.25 90))
-    (property "Footprint" "" (id 2) (at 91.44 99.06 0)
+    (property "Footprint" "SnapEDA Library:WSKW06122L000FEA" (id 2) (at 91.44 99.06 0)
       (effects (font (size 1.27 1.27)) hide)
     )
@@
       (effects (font (size 1.27 1.27)) (justify left))
     )
-    (property "Footprint" "" (id 2) (at 147.32 25.4 0)
+    (property "Footprint" "Capacitor_SMD:C_0805_2012Metric_Pad1.18x1.45mm_HandSolder" (id 2) (at 147.32 25.4 0)
       (effects (font (size 1.27 1.27)) hide)
     )
@@
       (effects (font (size 1.27 1.27)) (justify left))
     )
-    (property "Footprint" "" (id 2) (at 205.74 63.5 0)
+    (property "Footprint" "Capacitor_SMD:C_0805_2012Metric_Pad1.18x1.45mm_HandSolder" (id 2) (at 205.74 63.5 0)
       (effects (font (size 1.27 1.27)) hide)
     )
@@
     (property "Reference" "R13" (id 0) (at 193.04 36.83 90))
     (property "Value" "2m" (id 1) (at 193.04 39.37 90))
-    (property "Footprint" "" (id 2) (at 193.04 43.18 0)
+    (property "Footprint" "SnapEDA Library:WSKW06122L000FEA" (id 2) (at 193.04 43.18 0)
       (effects (font (size 1.27 1.27)) hide)
     )
@@
     (property "Reference" "U8" (id 0) (at 160.02 30.48 0))
     (property "Value" "EPC2152" (id 1) (at 160.02 33.02 0))
-    (property "Footprint" "" (id 2) (at 163.195 31.75 0)
+    (property "Footprint" "SnapEDA Library:EPC2152" (id 2) (at 163.195 31.75 0)
       (effects (font (size 1.27 1.27)) hide)
     )
@@
       (effects (font (size 1.27 1.27)) (justify left))
     )
-    (property "Footprint" "" (id 2) (at 45.72 88.9 0)
+    (property "Footprint" "Capacitor_SMD:C_0805_2012Metric_Pad1.18x1.45mm_HandSolder" (id 2) (at 45.72 88.9 0)
       (effects (font (size 1.27 1.27)) hide)
     )
@@
       (effects (font (size 1.27 1.27)) (justify left))
     )
-    (property "Footprint" "" (id 2) (at 104.14 119.38 0)
+    (property "Footprint" "Capacitor_SMD:C_0805_2012Metric_Pad1.18x1.45mm_HandSolder" (id 2) (at 104.14 119.38 0)
       (effects (font (size 1.27 1.27)) hide)
     )
@@
     (property "Reference" "U5" (id 0) (at 58.42 86.36 0))
     (property "Value" "EPC2152" (id 1) (at 58.42 88.9 0))
-    (property "Footprint" "" (id 2) (at 61.595 87.63 0)
+    (property "Footprint" "SnapEDA Library:EPC2152" (id 2) (at 61.595 87.63 0)
       (effects (font (size 1.27 1.27)) hide)
     )
@@
       (effects (font (size 1.27 1.27)) (justify left))
     )
-    (property "Footprint" "" (id 2) (at 104.14 63.5 0)
+    (property "Footprint" "Capacitor_SMD:C_0805_2012Metric_Pad1.18x1.45mm_HandSolder" (id 2) (at 104.14 63.5 0)
       (effects (font (size 1.27 1.27)) hide)
     )
@@
       (effects (font (size 1.27 1.27)) (justify left))
     )
-    (property "Footprint" "" (id 2) (at 45.72 33.02 0)
+    (property "Footprint" "Capacitor_SMD:C_0805_2012Metric_Pad1.18x1.45mm_HandSolder" (id 2) (at 45.72 33.02 0)
       (effects (font (size 1.27 1.27)) hide)
     )
@@
     (property "Reference" "U6" (id 0) (at 91.44 45.72 0))
     (property "Value" "INA181A2IDBVT" (id 1) (at 91.44 48.26 0))
-    (property "Footprint" "" (id 2) (at 91.44 63.5 0)
-      (effects (font (size 1.27 1.27)) hide)
-    )
+    (property "Footprint" "Package_TO_SOT_SMD:SOT-23-6_Handsoldering" (id 2) (at 91.44 63.5 0)
+      (effects (font (size 1.27 1.27)) hide)
+    )

Commit message: microcontroller done?
Parts:
- renumbered C20 to C22, C21 to C23, C22 to C24, C23 to C25, C24 to C26, C25 to C27, C26 to C28, C27 to C29, C28 to C30, R8 to R11, R9 to R12, R10 to R13, R11 to R14, R12 to R15, R13 to R16

Commit message: Net changes, sense changes
Connections:
- net VCC renamed VS
- net VDD renamed +12V
Changed lines of the file:
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@@
     (pin "1")
   )
-  (symbol (lib_id "power:VDD") (at 137.16 20.32 0) (unit 1)
-    (in_bom yes) (on_board yes) (fields_autoplaced)
-    (property "Reference" "#PWR040" (id 0) (at 137.16 24.13 0)
-      (effects (font (size 1.27 1.27)) hide)
-    )
-    (property "Value" "VDD" (id 1) (at 137.16 15.24 0))
+  (symbol (lib_id "power:+12V") (at 137.16 20.32 0) (unit 1)
+    (in_bom yes) (on_board yes) (fields_autoplaced)
+    (property "Reference" "#PWR?" (id 0) (at 137.16 24.13 0)
+      (effects (font (size 1.27 1.27)) hide)
+    )
+    (property "Value" "+12V" (id 1) (at 137.16 15.24 0))
     (property "Footprint" "" (id 2) (at 137.16 20.32 0)
       (effects (font (size 1.27 1.27)) hide)
@@
     (pin "6")
   )
-  (symbol (lib_id "power:VDD") (at 35.56 76.2 0) (unit 1)
-    (in_bom yes) (on_board yes) (fields_autoplaced)
-    (property "Reference" "#PWR026" (id 0) (at 35.56 80.01 0)
-      (effects (font (size 1.27 1.27)) hide)
-    )
-    (property "Value" "VDD" (id 1) (at 35.56 71.12 0))
-    (property "Footprint" "" (id 2) (at 35.56 76.2 0)
-      (effects (font (size 1.27 1.27)) hide)
-    )
-    (property "Datasheet" "" (id 3) (at 35.56 76.2 0)
-      (effects (font (size 1.27 1.27)) hide)
-    )
-    (pin "1")
-  )
   (symbol (lib_id "INA181A2IDBVT:INA181A2IDBVT") (at 91.44 119.38 0) (mirror x) (unit 1)
     (in_bom yes) (on_board yes) (fields_autoplaced)
@@
     (pin "1")
   )
+  (symbol (lib_id "power:VS") (at 167.64 30.48 0) (unit 1)
+    (in_bom yes) (on_board yes) (fields_autoplaced)
+    (property "Reference" "#PWR?" (id 0) (at 162.56 34.29 0)
+      (effects (font (size 1.27 1.27)) hide)
+    )
+    (property "Value" "VS" (id 1) (at 167.64 25.4 0))
+    (property "Footprint" "" (id 2) (at 167.64 30.48 0)
+      (effects (font (size 1.27 1.27)) hide)
+    )
+    (property "Datasheet" "" (id 3) (at 167.64 30.48 0)
+      (effects (font (size 1.27 1.27)) hide)
+    )
+    (pin "1")
+  )
+  (symbol (lib_id "power:VS") (at 66.04 30.48 0) (unit 1)
+    (in_bom yes) (on_board yes) (fields_autoplaced)
+    (property "Reference" "#PWR?" (id 0) (at 60.96 34.29 0)
+      (effects (font (size 1.27 1.27)) hide)
+    )
+    (property "Value" "" (id 1) (at 66.04 25.4 0))
+    (property "Footprint" "" (id 2) (at 66.04 30.48 0)
+      (effects (font (size 1.27 1.27)) hide)
+    )
+    (property "Datasheet" "" (id 3) (at 66.04 30.48 0)
+      (effects (font (size 1.27 1.27)) hide)
+    )
+    (pin "1")
+  )
   (symbol (lib_id "power:GND") (at 104.14 124.46 0) (unit 1)
     (in_bom yes) (on_board yes) (fields_autoplaced)
@@
     )
     (property "Datasheet" "" (id 3) (at 180.34 58.42 0)
+      (effects (font (size 1.27 1.27)) hide)
+    )
+    (pin "1")
+  )
+  (symbol (lib_id "power:VS") (at 66.04 86.36 0) (unit 1)
+    (in_bom yes) (on_board yes) (fields_autoplaced)
+    (property "Reference" "#PWR?" (id 0) (at 60.96 90.17 0)
+      (effects (font (size 1.27 1.27)) hide)
+    )
+    (property "Value" "VS" (id 1) (at 66.04 81.28 0))
+    (property "Footprint" "" (id 2) (at 66.04 86.36 0)
+      (effects (font (size 1.27 1.27)) hide)
+    )
+    (property "Datasheet" "" (id 3) (at 66.04 86.36 0)
       (effects (font (size 1.27 1.27)) hide)
     )
@@
     (pin "1")
   )
-  (symbol (lib_id "power:VCC") (at 66.04 86.36 0) (unit 1)
-    (in_bom yes) (on_board yes) (fields_autoplaced)
-    (property "Reference" "#PWR029" (id 0) (at 66.04 90.17 0)
-      (effects (font (size 1.27 1.27)) hide)
-    )
-    (property "Value" "VCC" (id 1) (at 66.04 81.28 0))
-    (property "Footprint" "" (id 2) (at 66.04 86.36 0)
-      (effects (font (size 1.27 1.27)) hide)
-    )
-    (property "Datasheet" "" (id 3) (at 66.04 86.36 0)
-      (effects (font (size 1.27 1.27)) hide)
-    )
-    (pin "1")
-  )
   (symbol (lib_id "Device:C_Small") (at 25.4 86.36 0) (unit 1)
     (in_bom yes) (on_board yes) (fields_autoplaced)
@@
     (pin "1")
     (pin "2")
-  )
-  (symbol (lib_id "power:VCC") (at 66.04 30.48 0) (unit 1)
-    (in_bom yes) (on_board yes) (fields_autoplaced)
-    (property "Reference" "#PWR027" (id 0) (at 66.04 34.29 0)
-      (effects (font (size 1.27 1.27)) hide)
-    )
-    (property "Value" "VCC" (id 1) (at 66.04 25.4 0))
-    (property "Footprint" "" (id 2) (at 66.04 30.48 0)
-      (effects (font (size 1.27 1.27)) hide)
-    )
-    (property "Datasheet" "" (id 3) (at 66.04 30.48 0)
-      (effects (font (size 1.27 1.27)) hide)
-    )
-    (pin "1")
   )
   (symbol (lib_id "Device:R_Small_US") (at 91.44 99.06 90) (unit 1)
@@
     )
     (property "Datasheet" "" (id 3) (at 127 35.56 0)
+      (effects (font (size 1.27 1.27)) hide)
+    )
+    (pin "1")
+  )
+  (symbol (lib_id "power:+12V") (at 35.56 20.32 0) (unit 1)
+    (in_bom yes) (on_board yes) (fields_autoplaced)
+    (property "Reference" "#PWR?" (id 0) (at 35.56 24.13 0)
+      (effects (font (size 1.27 1.27)) hide)
+    )
+    (property "Value" "" (id 1) (at 35.56 15.24 0))
+    (property "Footprint" "" (id 2) (at 35.56 20.32 0)
+      (effects (font (size 1.27 1.27)) hide)
+    )
+    (property "Datasheet" "" (id 3) (at 35.56 20.32 0)
       (effects (font (size 1.27 1.27)) hide)
     )
@@
     (pin "7")
   )
+  (symbol (lib_id "power:+12V") (at 35.56 76.2 0) (unit 1)
+    (in_bom yes) (on_board yes) (fields_autoplaced)
+    (property "Reference" "#PWR?" (id 0) (at 35.56 80.01 0)
+      (effects (font (size 1.27 1.27)) hide)
+    )
+    (property "Value" "+12V" (id 1) (at 35.56 71.12 0))
+    (property "Footprint" "" (id 2) (at 35.56 76.2 0)
+      (effects (font (size 1.27 1.27)) hide)
+    )
+    (property "Datasheet" "" (id 3) (at 35.56 76.2 0)
+      (effects (font (size 1.27 1.27)) hide)
+    )
+    (pin "1")
+  )
   (symbol (lib_id "power:GND") (at 205.74 68.58 0) (unit 1)
     (in_bom yes) (on_board yes) (fields_autoplaced)
@@
     (pin "2")
   )
-  (symbol (lib_id "power:VCC") (at 167.64 30.48 0) (unit 1)
-    (in_bom yes) (on_board yes) (fields_autoplaced)
-    (property "Reference" "#PWR041" (id 0) (at 167.64 34.29 0)
-      (effects (font (size 1.27 1.27)) hide)
-    )
-    (property "Value" "VCC" (id 1) (at 167.64 25.4 0))
-    (property "Footprint" "" (id 2) (at 167.64 30.48 0)
-      (effects (font (size 1.27 1.27)) hide)
-    )
-    (property "Datasheet" "" (id 3) (at 167.64 30.48 0)
-      (effects (font (size 1.27 1.27)) hide)
-    )
-    (pin "1")
-  )
   (symbol (lib_id "Device:R_Small_US") (at 45.72 33.02 0) (unit 1)
     (in_bom yes) (on_board yes) (fields_autoplaced)
@@
     (pin "2")
   )
-  (symbol (lib_id "power:VDD") (at 35.56 20.32 0) (unit 1)
-    (in_bom yes) (on_board yes) (fields_autoplaced)
-    (property "Reference" "#PWR025" (id 0) (at 35.56 24.13 0)
-      (effects (font (size 1.27 1.27)) hide)
-    )
-    (property "Value" "VDD" (id 1) (at 35.56 15.24 0))
-    (property "Footprint" "" (id 2) (at 35.56 20.32 0)
-      (effects (font (size 1.27 1.27)) hide)
-    )
-    (property "Datasheet" "" (id 3) (at 35.56 20.32 0)
-      (effects (font (size 1.27 1.27)) hide)
-    )
-    (pin "1")
-  )
   (symbol (lib_id "INA181A2IDBVT:INA181A2IDBVT") (at 91.44 63.5 0) (mirror x) (unit 1)
