File: hardware/microcontroller.kicad_sch (KiCad schematic)
At the start: 13 parts, among them SW1 SW_DPST, U1 ATSAMD21G18A-M, Y1 Crystal

Commit message: signal leds, bulk capacitance
Other:
- note added: "please assign analog pin for phase sense."
Changed lines of the file:
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@@
   (no_connect (at 76.2 114.3))
   (no_connect (at 76.2 116.84))
+  (polyline (pts (xy 91.44 85.09) (xy 91.44 76.2))
+    (stroke (width 0) (type default) (color 0 0 0 0))
+  )
   (wire (pts (xy 132.08 31.75) (xy 143.51 31.75))
     (stroke (width 0) (type default) (color 0 0 0 0))
@@
     (stroke (width 0) (type default) (color 0 0 0 0))
   )
+  (polyline (pts (xy 63.5 76.2) (xy 46.99 76.2))
+    (stroke (width 0) (type default) (color 0 0 0 0))
+  )
   (wire (pts (xy 142.24 53.34) (xy 147.32 53.34))
     (stroke (width 0) (type default) (color 0 0 0 0))
@@
   )
   (wire (pts (xy 143.51 24.13) (xy 154.94 24.13))
+    (stroke (width 0) (type default) (color 0 0 0 0))
+  )
+  (polyline (pts (xy 46.99 76.2) (xy 46.99 85.09))
     (stroke (width 0) (type default) (color 0 0 0 0))
   )
@@
     (stroke (width 0) (type default) (color 0 0 0 0))
   )
+  (polyline (pts (xy 46.99 85.09) (xy 91.44 85.09))
+    (stroke (width 0) (type default) (color 0 0 0 0))
+  )
   (wire (pts (xy 107.95 52.07) (xy 116.84 52.07))
     (stroke (width 0) (type default) (color 0 0 0 0))
@@
     (stroke (width 0) (type default) (color 0 0 0 0))
   )
+  (polyline (pts (xy 63.5 76.2) (xy 91.44 76.2))
+    (stroke (width 0) (type default) (color 0 0 0 0))
+  )
   (wire (pts (xy 137.16 149.86) (xy 139.7 149.86))
     (stroke (width 0) (type default) (color 0 0 0 0))
@@
   )
   (text "17" (at 143.51 24.13 0)
+    (effects (font (size 1.27 1.27)) (justify left bottom))
+  )
+  (text "please assign analog pin for phase sense." (at 48.26 78.74 0)
     (effects (font (size 1.27 1.27)) (justify left bottom))
   )
@@
       (effects (font (size 1.27 1.27)) (justify right) hide)
     )
+  )
+  (global_label "VSNS_W" (shape input) (at 78.74 82.55 180) (fields_autoplaced)
+    (effects (font (size 1.27 1.27)) (justify right))
+    (property "Intersheet References" "${INTERSHEET_REFS}" (id 0) (at 69.0698 82.6294 0)
+      (effects (font (size 1.27 1.27)) (justify right) hide)
+    )
