File: hardware/sense.kicad_sch (KiCad schematic)
At the start: 0 parts

Commit message: added buck converter rev1
still need to pick inductors, size bulk capacitance, verify calcs
Parts:
- added R? (x3): 10k, symbol Device:R_Small_US
- added R? (x3): 175k, symbol Device:R_Small_US
Connections:
- new net: R?.2, R?.2, R?.2
- new net PH_A: R?.1
- new net PH_B: R?.1
- new net PH_C: R?.1
- new net V_AN: R?.1, R?.2
- new net V_CN: R?.1, R?.1, R?.2, R?.2
Other:
- note added: "Should provide 3.25V @60V pk"
Changed lines of the file:
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@@
 (kicad_sch (version 20211123) (generator eeschema)
   (paper "A4")
+  (junction (at 101.6 48.26) (diameter 0) (color 0 0 0 0)
+  )
+  (junction (at 76.2 48.26) (diameter 0) (color 0 0 0 0)
+  )
+  (junction (at 88.9 48.26) (diameter 0) (color 0 0 0 0)
+  )
+  (junction (at 88.9 35.56) (diameter 0) (color 0 0 0 0)
+  )
+  (wire (pts (xy 50.8 38.1) (xy 66.04 38.1))
+    (stroke (width 0) (type default) (color 0 0 0 0))
+  )
+  (wire (pts (xy 50.8 50.8) (xy 111.76 50.8))
+    (stroke (width 0) (type default) (color 0 0 0 0))
+  )
+  (wire (pts (xy 66.04 48.26) (xy 66.04 38.1))
+    (stroke (width 0) (type default) (color 0 0 0 0))
+  )
+  (wire (pts (xy 83.82 48.26) (xy 88.9 48.26))
+    (stroke (width 0) (type default) (color 0 0 0 0))
+  )
+  (wire (pts (xy 99.06 48.26) (xy 101.6 48.26))
+    (stroke (width 0) (type default) (color 0 0 0 0))
+  )
+  (wire (pts (xy 111.76 48.26) (xy 111.76 50.8))
+    (stroke (width 0) (type default) (color 0 0 0 0))
+  )
+  (wire (pts (xy 88.9 33.02) (xy 88.9 35.56))
+    (stroke (width 0) (type default) (color 0 0 0 0))
+  )
+  (wire (pts (xy 88.9 35.56) (xy 88.9 38.1))
+    (stroke (width 0) (type default) (color 0 0 0 0))
+  )
+  (wire (pts (xy 50.8 25.4) (xy 88.9 25.4))
+    (stroke (width 0) (type default) (color 0 0 0 0))
+  )
+  (wire (pts (xy 109.22 48.26) (xy 111.76 48.26))
+    (stroke (width 0) (type default) (color 0 0 0 0))
+  )
+  (wire (pts (xy 101.6 48.26) (xy 104.14 48.26))
+    (stroke (width 0) (type default) (color 0 0 0 0))
+  )
+  (wire (pts (xy 76.2 35.56) (xy 76.2 48.26))
+    (stroke (width 0) (type default) (color 0 0 0 0))
+  )
+  (wire (pts (xy 88.9 48.26) (xy 88.9 43.18))
+    (stroke (width 0) (type default) (color 0 0 0 0))
+  )
+  (wire (pts (xy 73.66 48.26) (xy 76.2 48.26))
+    (stroke (width 0) (type default) (color 0 0 0 0))
+  )
+  (wire (pts (xy 73.66 35.56) (xy 76.2 35.56))
+    (stroke (width 0) (type default) (color 0 0 0 0))
+  )
+  (wire (pts (xy 76.2 48.26) (xy 78.74 48.26))
+    (stroke (width 0) (type default) (color 0 0 0 0))
+  )
+  (wire (pts (xy 101.6 38.1) (xy 101.6 48.26))
+    (stroke (width 0) (type default) (color 0 0 0 0))
+  )
+  (wire (pts (xy 88.9 35.56) (xy 91.44 35.56))
+    (stroke (width 0) (type default) (color 0 0 0 0))
+  )
+  (wire (pts (xy 88.9 27.94) (xy 88.9 25.4))
+    (stroke (width 0) (type default) (color 0 0 0 0))
+  )
+  (wire (pts (xy 68.58 48.26) (xy 66.04 48.26))
+    (stroke (width 0) (type default) (color 0 0 0 0))
+  )
+  (wire (pts (xy 104.14 38.1) (xy 101.6 38.1))
+    (stroke (width 0) (type default) (color 0 0 0 0))
+  )
+  (wire (pts (xy 93.98 48.26) (xy 88.9 48.26))
+    (stroke (width 0) (type default) (color 0 0 0 0))
+  )
+  (text "Should provide 3.25V @60V pk" (at 71.12 20.32 0)
+    (effects (font (size 1.27 1.27)) (justify left bottom))
+  )
+  (global_label "V_AN" (shape input) (at 91.44 35.56 0) (fields_autoplaced)
+    (effects (font (size 1.27 1.27)) (justify left))
+    (property "Intersheet References" "${INTERSHEET_REFS}" (id 0) (at 98.3283 35.4806 0)
+      (effects (font (size 1.27 1.27)) (justify left) hide)
+    )
+  )
+  (global_label "V_CN" (shape input) (at 73.66 35.56 180) (fields_autoplaced)
+    (effects (font (size 1.27 1.27)) (justify right))
+    (property "Intersheet References" "${INTERSHEET_REFS}" (id 0) (at 66.5902 35.4806 0)
+      (effects (font (size 1.27 1.27)) (justify right) hide)
+    )
+  )
+  (global_label "PH_B" (shape input) (at 50.8 38.1 180) (fields_autoplaced)
+    (effects (font (size 1.27 1.27)) (justify right))
+    (property "Intersheet References" "${INTERSHEET_REFS}" (id 0) (at 43.5488 38.0206 0)
+      (effects (font (size 1.27 1.27)) (justify right) hide)
+    )
+  )
+  (global_label "PH_A" (shape input) (at 50.8 25.4 180) (fields_autoplaced)
+    (effects (font (size 1.27 1.27)) (justify right))
+    (property "Intersheet References" "${INTERSHEET_REFS}" (id 0) (at 43.7302 25.3206 0)
+      (effects (font (size 1.27 1.27)) (justify right) hide)
+    )
+  )
+  (global_label "V_CN" (shape input) (at 104.14 38.1 0) (fields_autoplaced)
+    (effects (font (size 1.27 1.27)) (justify left))
+    (property "Intersheet References" "${INTERSHEET_REFS}" (id 0) (at 111.2098 38.0206 0)
+      (effects (font (size 1.27 1.27)) (justify left) hide)
+    )
+  )
+  (global_label "PH_C" (shape input) (at 50.8 50.8 180) (fields_autoplaced)
+    (effects (font (size 1.27 1.27)) (justify right))
+    (property "Intersheet References" "${INTERSHEET_REFS}" (id 0) (at 43.5488 50.7206 0)
+      (effects (font (size 1.27 1.27)) (justify right) hide)
+    )
+  )
+  (symbol (lib_id "Device:R_Small_US") (at 88.9 40.64 0) (unit 1)
+    (in_bom yes) (on_board yes)
+    (property "Reference" "R?" (id 0) (at 91.44 38.1 0)
+      (effects (font (size 1.27 1.27)) (justify left))
+    )
+    (property "Value" "10k" (id 1) (at 91.44 40.64 0)
+      (effects (font (size 1.27 1.27)) (justify left))
+    )
+    (property "Footprint" "" (id 2) (at 88.9 40.64 0)
+      (effects (font (size 1.27 1.27)) hide)
+    )
+    (property "Datasheet" "~" (id 3) (at 88.9 40.64 0)
+      (effects (font (size 1.27 1.27)) hide)
+    )
+    (pin "1")
+    (pin "2")
+  )
+  (symbol (lib_id "Device:R_Small_US") (at 106.68 48.26 270) (unit 1)
+    (in_bom yes) (on_board yes)
+    (property "Reference" "R?" (id 0) (at 106.68 43.18 90)
+      (effects (font (size 1.27 1.27)) (justify left))
+    )
+    (property "Value" "175k" (id 1) (at 106.68 45.72 90)
+      (effects (font (size 1.27 1.27)) (justify left))
+    )
+    (property "Footprint" "" (id 2) (at 106.68 48.26 0)
+      (effects (font (size 1.27 1.27)) hide)
+    )
+    (property "Datasheet" "~" (id 3) (at 106.68 48.26 0)
+      (effects (font (size 1.27 1.27)) hide)
+    )
+    (pin "1")
+    (pin "2")
+  )
+  (symbol (lib_id "Device:R_Small_US") (at 96.52 48.26 270) (unit 1)
+    (in_bom yes) (on_board yes)
+    (property "Reference" "R?" (id 0) (at 96.52 43.18 90)
+      (effects (font (size 1.27 1.27)) (justify left))
+    )
+    (property "Value" "10k" (id 1) (at 96.52 45.72 90)
+      (effects (font (size 1.27 1.27)) (justify left))
+    )
+    (property "Footprint" "" (id 2) (at 96.52 48.26 0)
+      (effects (font (size 1.27 1.27)) hide)
+    )
+    (property "Datasheet" "~" (id 3) (at 96.52 48.26 0)
+      (effects (font (size 1.27 1.27)) hide)
+    )
+    (pin "1")
+    (pin "2")
+  )
+  (symbol (lib_id "Device:R_Small_US") (at 71.12 48.26 90) (unit 1)
+    (in_bom yes) (on_board yes)
+    (property "Reference" "R?" (id 0) (at 73.66 43.18 90)
+      (effects (font (size 1.27 1.27)) (justify left))
+    )
+    (property "Value" "175k" (id 1) (at 73.66 45.72 90)
+      (effects (font (size 1.27 1.27)) (justify left))
+    )
+    (property "Footprint" "" (id 2) (at 71.12 48.26 0)
+      (effects (font (size 1.27 1.27)) hide)
+    )
+    (property "Datasheet" "~" (id 3) (at 71.12 48.26 0)
+      (effects (font (size 1.27 1.27)) hide)
+    )
+    (pin "1")
+    (pin "2")
+  )
+  (symbol (lib_id "Device:R_Small_US") (at 81.28 48.26 90) (unit 1)
+    (in_bom yes) (on_board yes)
+    (property "Reference" "R?" (id 0) (at 82.55 45.7201 90)
+      (effects (font (size 1.27 1.27)) (justify left))
+    )
+    (property "Value" "10k" (id 1) (at 82.55 43.1801 90)
+      (effects (font (size 1.27 1.27)) (justify left))
+    )
+    (property "Footprint" "" (id 2) (at 81.28 48.26 0)
+      (effects (font (size 1.27 1.27)) hide)
+    )
+    (property "Datasheet" "~" (id 3) (at 81.28 48.26 0)
+      (effects (font (size 1.27 1.27)) hide)
+    )
+    (pin "1")
+    (pin "2")
+  )
+  (symbol (lib_id "Device:R_Small_US") (at 88.9 30.48 0) (unit 1)
+    (in_bom yes) (on_board yes) (fields_autoplaced)
+    (property "Reference" "R?" (id 0) (at 91.44 29.2099 0)
+      (effects (font (size 1.27 1.27)) (justify left))
+    )
+    (property "Value" "175k" (id 1) (at 91.44 31.7499 0)
+      (effects (font (size 1.27 1.27)) (justify left))
+    )
+    (property "Footprint" "" (id 2) (at 88.9 30.48 0)
+      (effects (font (size 1.27 1.27)) hide)
+    )
+    (property "Datasheet" "~" (id 3) (at 88.9 30.48 0)
+      (effects (font (size 1.27 1.27)) hide)
+    )
+    (pin "1")
+    (pin "2")
+  )
 )

Commit message: Started Buck Layout
Parts:
- gave numbers to parts that had none: 6
Other:
- note added: "to be updated, not final"
Changed lines of the file:
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@@
+    (effects (font (size 1.27 1.27)) (justify left bottom))
+  )
+  (text "to be updated, not final\n" (at 71.12 22.86 0)
     (effects (font (size 1.27 1.27)) (justify left bottom))
   )
@@
   (symbol (lib_id "Device:R_Small_US") (at 88.9 40.64 0) (unit 1)
     (in_bom yes) (on_board yes)
-    (property "Reference" "R?" (id 0) (at 91.44 38.1 0)
+    (property "Reference" "R17" (id 0) (at 91.44 38.1 0)
       (effects (font (size 1.27 1.27)) (justify left))
     )
@@
   (symbol (lib_id "Device:R_Small_US") (at 106.68 48.26 270) (unit 1)
     (in_bom yes) (on_board yes)
-    (property "Reference" "R?" (id 0) (at 106.68 43.18 90)
+    (property "Reference" "R19" (id 0) (at 106.68 43.18 90)
       (effects (font (size 1.27 1.27)) (justify left))
     )
@@
   (symbol (lib_id "Device:R_Small_US") (at 96.52 48.26 270) (unit 1)
     (in_bom yes) (on_board yes)
-    (property "Reference" "R?" (id 0) (at 96.52 43.18 90)
+    (property "Reference" "R18" (id 0) (at 96.52 43.18 90)
       (effects (font (size 1.27 1.27)) (justify left))
     )
@@
   (symbol (lib_id "Device:R_Small_US") (at 71.12 48.26 90) (unit 1)
     (in_bom yes) (on_board yes)
-    (property "Reference" "R?" (id 0) (at 73.66 43.18 90)
+    (property "Reference" "R14" (id 0) (at 73.66 43.18 90)
       (effects (font (size 1.27 1.27)) (justify left))
     )
@@
   (symbol (lib_id "Device:R_Small_US") (at 81.28 48.26 90) (unit 1)
     (in_bom yes) (on_board yes)
-    (property "Reference" "R?" (id 0) (at 82.55 45.7201 90)
+    (property "Reference" "R15" (id 0) (at 82.55 45.7201 90)
       (effects (font (size 1.27 1.27)) (justify left))
     )
@@
   (symbol (lib_id "Device:R_Small_US") (at 88.9 30.48 0) (unit 1)
     (in_bom yes) (on_board yes) (fields_autoplaced)
-    (property "Reference" "R?" (id 0) (at 91.44 29.2099 0)
+    (property "Reference" "R16" (id 0) (at 91.44 29.2099 0)
       (effects (font (size 1.27 1.27)) (justify left))
     )

Commit message: workin away
Parts:
- added U?: AS5048A, Package_SO:TSSOP-14_4.4x5mm_P0.65mm, symbol Sensor_Magnetic:AS5048A
Changed lines of the file:
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@@
     (pin "2")
+  )
+  (symbol (lib_id "Sensor_Magnetic:AS5048A") (at 85.09 90.17 0) (unit 1)
+    (in_bom yes) (on_board yes) (fields_autoplaced)
+    (property "Reference" "U?" (id 0) (at 100.33 85.8393 0))
+    (property "Value" "AS5048A" (id 1) (at 100.33 88.3793 0))
+    (property "Footprint" "Package_SO:TSSOP-14_4.4x5mm_P0.65mm" (id 2) (at 85.09 109.22 0)
+      (effects (font (size 1.27 1.27)) hide)
+    )
+    (property "Datasheet" "https://ams.com/documents/20143/36005/AS5048_DS000298_4-00.pdf" (id 3) (at 30.48 49.53 0)
+      (effects (font (size 1.27 1.27)) hide)
+    )
+    (pin "1")
+    (pin "10")
+    (pin "11")
+    (pin "12")
+    (pin "13")
+    (pin "14")
+    (pin "2")
+    (pin "3")
+    (pin "4")
+    (pin "5")
+    (pin "6")
+    (pin "7")
+    (pin "8")
+    (pin "9")
   )
   (symbol (lib_id "Device:R_Small_US") (at 81.28 48.26 90) (unit 1)

Commit message: microcontroller done?
Parts:
- added C31: 100n, Capacitor_SMD:C_0402_1005Metric, symbol Device:C
- added C32: 10u, Capacitor_SMD:C_0805_2012Metric, symbol Device:C
- gave numbers to parts that had none: 1
- renumbered R14 to R17, R15 to R18, R16 to R19, R17 to R20, R18 to R21, R19 to R22
Connections:
- net CS_ENC: now reaches U10.1 (~{CSn})
- net at U10.11 (VDD5V): now also U10.12 (VDD3V), C31.1, C32.1
- net SCK: now reaches U10.2 (CLK)
- net MISO: now reaches U10.3 (MISO)
- net MOSI: now reaches U10.4 (MOSI)
- new net GND: C31.2, C32.2
- no-connect marks 0 -> 7
Other:
- moved on the sheet: U10
Changed lines of the file:
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@@
 (kicad_sch (version 20211123) (generator eeschema)
   (paper "A4")
+  (junction (at 81.28 66.04) (diameter 0) (color 0 0 0 0)
+  )
   (junction (at 101.6 48.26) (diameter 0) (color 0 0 0 0)
   )
+  (junction (at 76.2 76.2) (diameter 0) (color 0 0 0 0)
+  )
   (junction (at 76.2 48.26) (diameter 0) (color 0 0 0 0)
   )
@@
   (junction (at 88.9 35.56) (diameter 0) (color 0 0 0 0)
   )
+  (junction (at 93.98 73.66) (diameter 0) (color 0 0 0 0)
+  )
+  (no_connect (at 88.9 88.9))
+  (no_connect (at 81.28 101.6))
+  (no_connect (at 78.74 101.6))
+  (no_connect (at 76.2 101.6))
+  (no_connect (at 73.66 101.6))
+  (no_connect (at 71.12 101.6))
+  (no_connect (at 68.58 101.6))
   (wire (pts (xy 50.8 38.1) (xy 66.04 38.1))
     (stroke (width 0) (type default) (color 0 0 0 0))
@@
     (stroke (width 0) (type default) (color 0 0 0 0))
   )
+  (wire (pts (xy 81.28 73.66) (xy 93.98 73.66))
+    (stroke (width 0) (type default) (color 0 0 0 0))
+  )
   (wire (pts (xy 66.04 48.26) (xy 66.04 38.1))
     (stroke (width 0) (type default) (color 0 0 0 0))
@@
     (stroke (width 0) (type default) (color 0 0 0 0))
   )
+  (wire (pts (xy 76.2 66.04) (xy 81.28 66.04))
+    (stroke (width 0) (type default) (color 0 0 0 0))
+  )
+  (wire (pts (xy 73.66 76.2) (xy 76.2 76.2))
+    (stroke (width 0) (type default) (color 0 0 0 0))
+  )
   (wire (pts (xy 76.2 48.26) (xy 78.74 48.26))
     (stroke (width 0) (type default) (color 0 0 0 0))
   )
+  (wire (pts (xy 81.28 66.04) (xy 93.98 66.04))
+    (stroke (width 0) (type default) (color 0 0 0 0))
+  )
   (wire (pts (xy 101.6 38.1) (xy 101.6 48.26))
     (stroke (width 0) (type default) (color 0 0 0 0))
@@
   )
   (wire (pts (xy 68.58 48.26) (xy 66.04 48.26))
+    (stroke (width 0) (type default) (color 0 0 0 0))
+  )
+  (wire (pts (xy 76.2 76.2) (xy 76.2 66.04))
     (stroke (width 0) (type default) (color 0 0 0 0))
   )
@@
   (text "to be updated, not final\n" (at 71.12 22.86 0)
     (effects (font (size 1.27 1.27)) (justify left bottom))
+  )
+  (global_label "MISO" (shape input) (at 63.5 83.82 180) (fields_autoplaced)
+    (effects (font (size 1.27 1.27)) (justify right))
+    (property "Intersheet References" "${INTERSHEET_REFS}" (id 0) (at 56.4907 83.7406 0)
+      (effects (font (size 1.27 1.27)) (justify right) hide)
+    )
   )
   (global_label "V_AN" (shape input) (at 91.44 35.56 0) (fields_autoplaced)
@@
     )
   )
+  (global_label "SCK" (shape input) (at 63.5 86.36 180) (fields_autoplaced)
+    (effects (font (size 1.27 1.27)) (justify right))
+    (property "Intersheet References" "${INTERSHEET_REFS}" (id 0) (at 57.3374 86.2806 0)
+      (effects (font (size 1.27 1.27)) (justify right) hide)
+    )
+  )
   (global_label "PH_B" (shape input) (at 50.8 38.1 180) (fields_autoplaced)
     (effects (font (size 1.27 1.27)) (justify right))
     (property "Intersheet References" "${INTERSHEET_REFS}" (id 0) (at 43.5488 38.0206 0)
+      (effects (font (size 1.27 1.27)) (justify right) hide)
+    )
+  )
+  (global_label "CS_ENC" (shape input) (at 63.5 88.9 180) (fields_autoplaced)
+    (effects (font (size 1.27 1.27)) (justify right))
+    (property "Intersheet References" "${INTERSHEET_REFS}" (id 0) (at 53.8902 88.8206 0)
+      (effects (font (size 1.27 1.27)) (justify right) hide)
+    )
+  )
+  (global_label "MOSI" (shape input) (at 63.5 81.28 180) (fields_autoplaced)
+    (effects (font (size 1.27 1.27)) (justify right))
+    (property "Intersheet References" "${INTERSHEET_REFS}" (id 0) (at 56.4907 81.2006 0)
       (effects (font (size 1.27 1.27)) (justify right) hide)
     )
@@
     )
   )
+  (symbol (lib_id "Device:C") (at 93.98 69.85 0) (unit 1)
+    (in_bom yes) (on_board yes) (fields_autoplaced)
+    (property "Reference" "C32" (id 0) (at 97.79 68.5799 0)
+      (effects (font (size 1.27 1.27)) (justify left))
+    )
+    (property "Value" "10u" (id 1) (at 97.79 71.1199 0)
+      (effects (font (size 1.27 1.27)) (justify left))
+    )
+    (property "Footprint" "Capacitor_SMD:C_0805_2012Metric" (id 2) (at 94.9452 73.66 0)
+      (effects (font (size 1.27 1.27)) hide)
+    )
+    (property "Datasheet" "~" (id 3) (at 93.98 69.85 0)
+      (effects (font (size 1.27 1.27)) hide)
+    )
+    (property "Mouser" "https://www.mouser.com/ProductDetail/Murata-Electronics/GRM21BR61E106KA73K?qs=sGAEpiMZZMvsSlwiRhF8qtKev7nvVKumSMGXtfW0ekhTExf3kTusQw%3D%3D" (id 4) (at 93.98 69.85 0)
+      (effects (font (size 1.27 1.27)) hide)
+    )
+    (pin "1")
+    (pin "2")
+  )
   (symbol (lib_id "Device:R_Small_US") (at 88.9 40.64 0) (unit 1)
     (in_bom yes) (on_board yes)
-    (property "Reference" "R17" (id 0) (at 91.44 38.1 0)
+    (property "Reference" "R20" (id 0) (at 91.44 38.1 0)
       (effects (font (size 1.27 1.27)) (justify left))
     )
@@
   (symbol (lib_id "Device:R_Small_US") (at 106.68 48.26 270) (unit 1)
     (in_bom yes) (on_board yes)
-    (property "Reference" "R19" (id 0) (at 106.68 43.18 90)
+    (property "Reference" "R22" (id 0) (at 106.68 43.18 90)
       (effects (font (size 1.27 1.27)) (justify left))
     )
@@
   (symbol (lib_id "Device:R_Small_US") (at 96.52 48.26 270) (unit 1)
     (in_bom yes) (on_board yes)
-    (property "Reference" "R18" (id 0) (at 96.52 43.18 90)
+    (property "Reference" "R21" (id 0) (at 96.52 43.18 90)
       (effects (font (size 1.27 1.27)) (justify left))
     )
@@
     (pin "2")
   )
+  (symbol (lib_id "power:GND") (at 93.98 73.66 0) (unit 1)
+    (in_bom yes) (on_board yes) (fields_autoplaced)
+    (property "Reference" "#PWR047" (id 0) (at 93.98 80.01 0)
+      (effects (font (size 1.27 1.27)) hide)
+    )
+    (property "Value" "GND" (id 1) (at 93.98 78.74 0))
+    (property "Footprint" "" (id 2) (at 93.98 73.66 0)
+      (effects (font (size 1.27 1.27)) hide)
+    )
+    (property "Datasheet" "" (id 3) (at 93.98 73.66 0)
+      (effects (font (size 1.27 1.27)) hide)
+    )
+    (pin "1")
+  )
+  (symbol (lib_id "Device:C") (at 81.28 69.85 0) (unit 1)
+    (in_bom yes) (on_board yes) (fields_autoplaced)
+    (property "Reference" "C31" (id 0) (at 85.09 68.5799 0)
+      (effects (font (size 1.27 1.27)) (justify left))
+    )
+    (property "Value" "100n" (id 1) (at 85.09 71.1199 0)
+      (effects (font (size 1.27 1.27)) (justify left))
+    )
+    (property "Footprint" "Capacitor_SMD:C_0402_1005Metric" (id 2) (at 82.2452 73.66 0)
+      (effects (font (size 1.27 1.27)) hide)
+    )
+    (property "Datasheet" "~" (id 3) (at 81.28 69.85 0)
+      (effects (font (size 1.27 1.27)) hide)
+    )
+    (property "Mouser" "https://www.mouser.com/ProductDetail/Murata-Electronics/GCM155R71E104KE02D?qs=sGAEpiMZZMvsSlwiRhF8qsL%2Fc0EXNue%2FoQ0bAUFzBJynJfbvKN%252BGCA%3D%3D" (id 4) (at 81.28 69.85 0)
+      (effects (font (size 1.27 1.27)) hide)
+    )
+    (pin "1")
+    (pin "2")
+  )
   (symbol (lib_id "Device:R_Small_US") (at 71.12 48.26 90) (unit 1)
     (in_bom yes) (on_board yes)
-    (property "Reference" "R14" (id 0) (at 73.66 43.18 90)
+    (property "Reference" "R17" (id 0) (at 73.66 43.18 90)
       (effects (font (size 1.27 1.27)) (justify left))
     )
@@
     (pin "2")
   )
-  (symbol (lib_id "Sensor_Magnetic:AS5048A") (at 85.09 90.17 0) (unit 1)
-    (in_bom yes) (on_board yes) (fields_autoplaced)
-    (property "Reference" "U?" (id 0) (at 100.33 85.8393 0))
-    (property "Value" "AS5048A" (id 1) (at 100.33 88.3793 0))
-    (property "Footprint" "Package_SO:TSSOP-14_4.4x5mm_P0.65mm" (id 2) (at 85.09 109.22 0)
-      (effects (font (size 1.27 1.27)) hide)
-    )
-    (property "Datasheet" "https://ams.com/documents/20143/36005/AS5048_DS000298_4-00.pdf" (id 3) (at 30.48 49.53 0)
+  (symbol (lib_id "Sensor_Magnetic:AS5048A") (at 76.2 88.9 0) (unit 1)
+    (in_bom yes) (on_board yes) (fields_autoplaced)
+    (property "Reference" "U10" (id 0) (at 91.44 84.5693 0))
+    (property "Value" "AS5048A" (id 1) (at 91.44 87.1093 0))
+    (property "Footprint" "Package_SO:TSSOP-14_4.4x5mm_P0.65mm" (id 2) (at 76.2 107.95 0)
+      (effects (font (size 1.27 1.27)) hide)
+    )
+    (property "Datasheet" "https://ams.com/documents/20143/36005/AS5048_DS000298_4-00.pdf" (id 3) (at 21.59 48.26 0)
       (effects (font (size 1.27 1.27)) hide)
     )
@@
   (symbol (lib_id "Device:R_Small_US") (at 81.28 48.26 90) (unit 1)
     (in_bom yes) (on_board yes)
-    (property "Reference" "R15" (id 0) (at 82.55 45.7201 90)
+    (property "Reference" "R18" (id 0) (at 82.55 45.7201 90)
       (effects (font (size 1.27 1.27)) (justify left))
     )
@@
   (symbol (lib_id "Device:R_Small_US") (at 88.9 30.48 0) (unit 1)
     (in_bom yes) (on_board yes) (fields_autoplaced)
-    (property "Reference" "R16" (id 0) (at 91.44 29.2099 0)
-      (effects (font (size 1.27 1.27)) (justify left))
-    )
+    (property "Reference" "R19" (id 0) (at 91.44 29.2099 0)
+      (effects (font (size 1.27 1.27)) (justify left))
+    )

Commit message: Net changes, sense changes
Parts:
- removed R17, R19, R22: 175k, symbol Device:R_Small_US
- removed R18, R20, R21: 10k, symbol Device:R_Small_US
- added R? (x2): (no value), Resistor_SMD:R_0805_2012Metric, symbol Device:R_US
- added R?: 2Meg, Resistor_SMD:R_0805_2012Metric, symbol Device:R_US
- added R?: 10k, Resistor_SMD:R_0805_2012Metric, symbol Device:R_Small_US
- added U? (x3): (no value), symbol Device:Opamp_Dual
Connections:
- net GND: now also R?.1, U?.4 (V-)
- net PH_A: now also R?.1, R?.2, U?.1
- new net: R?.1, R?.2, U?.3 (+)
- new net: R?.1, R?.2, U?.2 (-)
- new net +12V: U?.8 (V+)
- new net VAA: R?.2
- no-connect marks 7 -> 10
Other:
- note removed: "to be updated, not final"
