File: hardware/sense.kicad_sch (KiCad schematic)
At the start: 10 parts, among them U10 AS5048A

Commit message: some layout
Parts:
- R28: renamed from R19; value 47k -> ~
- gave numbers to parts that had none: 2
- renumbered C31 to C51, C32 to C52, R18 to R27, R17 to R29, R20 to R30
Changed lines of the file:
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@@
   (symbol (lib_id "Device:R_US") (at 157.48 38.1 90) (unit 1)
     (in_bom yes) (on_board yes) (fields_autoplaced)
-    (property "Reference" "R18" (id 0) (at 157.48 31.75 90))
+    (property "Reference" "R27" (id 0) (at 157.48 31.75 90))
     (property "Value" "2Meg" (id 1) (at 157.48 34.29 90))
     (property "Footprint" "Resistor_SMD:R_0805_2012Metric" (id 2) (at 157.734 37.084 90)
@@
   (symbol (lib_id "power:+12V") (at 254 27.94 0) (unit 1)
     (in_bom yes) (on_board yes) (fields_autoplaced)
-    (property "Reference" "#PWR?" (id 0) (at 254 31.75 0)
+    (property "Reference" "#PWR067" (id 0) (at 254 31.75 0)
       (effects (font (size 1.27 1.27)) hide)
     )
@@
   (symbol (lib_id "power:GND") (at 154.94 45.72 0) (unit 1)
     (in_bom yes) (on_board yes) (fields_autoplaced)
-    (property "Reference" "#PWR047" (id 0) (at 154.94 52.07 0)
+    (property "Reference" "#PWR065" (id 0) (at 154.94 52.07 0)
       (effects (font (size 1.27 1.27)) hide)
     )
@@
   (symbol (lib_id "Device:C") (at 243.84 38.1 0) (mirror x) (unit 1)
     (in_bom yes) (on_board yes) (fields_autoplaced)
-    (property "Reference" "C?" (id 0) (at 240.03 36.8299 0)
+    (property "Reference" "C53" (id 0) (at 240.03 36.8299 0)
       (effects (font (size 1.27 1.27)) (justify right))
     )
@@
   (symbol (lib_id "Device:C") (at 93.98 69.85 0) (unit 1)
     (in_bom yes) (on_board yes) (fields_autoplaced)
-    (property "Reference" "C32" (id 0) (at 97.79 68.5799 0)
+    (property "Reference" "C52" (id 0) (at 97.79 68.5799 0)
       (effects (font (size 1.27 1.27)) (justify left))
     )
@@
   (symbol (lib_id "power:GND") (at 254 48.26 0) (unit 1)
     (in_bom yes) (on_board yes) (fields_autoplaced)
-    (property "Reference" "#PWR051" (id 0) (at 254 54.61 0)
+    (property "Reference" "#PWR068" (id 0) (at 254 54.61 0)
       (effects (font (size 1.27 1.27)) hide)
     )
@@
   (symbol (lib_id "Connector:TestPoint_Probe") (at 199.39 38.1 0) (unit 1)
     (in_bom yes) (on_board yes)
-    (property "Reference" "TP?" (id 0) (at 205.74 36.83 0)
+    (property "Reference" "TP4" (id 0) (at 205.74 36.83 0)
       (effects (font (size 1.27 1.27)) (justify right))
     )
@@
   (symbol (lib_id "Device:R_US") (at 171.45 43.18 90) (unit 1)
     (in_bom yes) (on_board yes)
-    (property "Reference" "R17" (id 0) (at 171.45 45.72 90))
+    (property "Reference" "R29" (id 0) (at 171.45 45.72 90))
     (property "Value" "2Meg" (id 1) (at 171.45 48.26 90))
     (property "Footprint" "Resistor_SMD:R_0805_2012Metric" (id 2) (at 171.704 42.164 90)
@@
   (symbol (lib_id "power:GND") (at 93.98 73.66 0) (unit 1)
     (in_bom yes) (on_board yes) (fields_autoplaced)
-    (property "Reference" "#PWR048" (id 0) (at 93.98 80.01 0)
+    (property "Reference" "#PWR064" (id 0) (at 93.98 80.01 0)
       (effects (font (size 1.27 1.27)) hide)
     )
@@
   (symbol (lib_id "Device:C") (at 81.28 69.85 0) (unit 1)
     (in_bom yes) (on_board yes) (fields_autoplaced)
-    (property "Reference" "C31" (id 0) (at 85.09 68.5799 0)
+    (property "Reference" "C51" (id 0) (at 85.09 68.5799 0)
       (effects (font (size 1.27 1.27)) (justify left))
     )
@@
   (symbol (lib_id "power:VAA") (at 165.1 22.86 0) (unit 1)
     (in_bom yes) (on_board yes) (fields_autoplaced)
-    (property "Reference" "#PWR049" (id 0) (at 165.1 26.67 0)
+    (property "Reference" "#PWR066" (id 0) (at 165.1 26.67 0)
       (effects (font (size 1.27 1.27)) hide)
     )
@@
   (symbol (lib_id "Device:R_Small_US") (at 189.23 50.8 90) (unit 1)
     (in_bom yes) (on_board yes)
-    (property "Reference" "R20" (id 0) (at 189.23 45.72 90))
+    (property "Reference" "R30" (id 0) (at 189.23 45.72 90))
     (property "Value" "10k" (id 1) (at 189.23 48.26 90))
     (property "Footprint" "Resistor_SMD:R_0805_2012Metric" (id 2) (at 189.23 50.8 0)
@@
   (symbol (lib_id "Device:R_US") (at 165.1 30.48 0) (mirror x) (unit 1)
     (in_bom yes) (on_board yes)
-    (property "Reference" "R19" (id 0) (at 168.91 29.21 0))
-    (property "Value" "47k" (id 1) (at 168.91 31.75 0))
+    (property "Reference" "R28" (id 0) (at 168.91 29.21 0))
+    (property "Value" "~" (id 1) (at 168.91 31.75 0))
     (property "Footprint" "Resistor_SMD:R_0805_2012Metric" (id 2) (at 166.116 30.226 90)
       (effects (font (size 1.27 1.27)) hide)

Commit message: Simplified sensing, added some power layout.
Parts:
- removed C53: 100n, Capacitor_SMD:C_0402_1005Metric, symbol Device:C
- removed R27: 2Meg, Resistor_SMD:R_0805_2012Metric, symbol Device:R_US
- removed R30: 10k, Resistor_SMD:R_0805_2012Metric, symbol Device:R_Small_US
- removed TP4: TestPoint_Probe, symbol Connector:TestPoint_Probe
- removed U11: ~, symbol Device:Opamp_Dual
- R28: value ~ -> 39k; Mouser https://www.mouser.com/ProductDetail/Panasonic/ERJ-6ENF5101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 -> (none)
- R29: value 2Meg -> 2.2k; Mouser https://www.mouser.com/ProductDetail/Panasonic/ERJ-6ENF5101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 -> (none)
- renumbered C51 to C53, C52 to C54, U10 to U9
Connections:
- net VAA is gone; now on net PH_W: R28.2
- net VSNS_W: now also R28.1, R29.2
- no-connect marks 10 -> 7
Other:
- note added: "I think I had this confused in my head, this should work."
- note removed: "Should provide 3.25Vp-p @60V p-p in biased to half scale"
